File: dev-board1/dev-board1.sch (EAGLE design)
At the start: 87 parts, among them IC1 MSP432E401, IC2 MT48LC16M16A2, IC3 SIM800C, IC4 CC3100MOD-LWK, IC5 TPD3E001DRL, IC6 TPD3E001DRL, IC7 TPD3E001DRL, J1 MAGJACK, J2 SIM-78723-1001, J3 ER-TFT024-3, J4 SWD_SHROUD, U3 ER-TFT024-3-OUTLINE, X2 BU-SMA-V

Commit message: adding power supply
Parts:
- added C39: 1u, passives-7351:CAPACITOR0603-N
- added C40: 47n, passives-7351:CAPACITOR0603-N
- added C41, C42, C44: 10u, passives-7351:CAPACITOR0805-N
- added C43: 4.7u, passives-7351:CAPACITOR0603-N
- added C45, C46, C47: 0805/10u/10V/X5R, TiLDA Mk3 Parts:C-EUC0805-N
- added IC8: BQ25601, TiLDA Mk4 Parts:BQ25601
- added IC9: TPS62082, TiLDA Mk3 Parts:TPS62082
- added JP2: (no value), TiLDA Mk4 Parts:M02-JST-2MM-SMT
- added L3: (no value), TiLDA Mk4 Parts:INDUCTOR1008
- added L4: SRN2512-2R2M, TiLDA Mk3 Parts:INDUCTOR1008
- added LED3: red, TiLDA Mk4 Parts:LED0603
- added Q6: CSD25402Q3A, TiLDA Mk3 Parts:CSD25402Q3A
- added R23, R25: 2k, passives-7351:RESISTOR0603-N
- added R24: dnp, passives-7351:RESISTOR0603-N
- added R26: 4.7k, passives-7351:RESISTOR0603-N
- added R27, R28: 10k, passives-7351:RESISTOR0603-N
- added R45: 0603/220k/5%, TiLDA Mk3 Parts:R-EU_0603K-SMALL
- added S3: (no value), Switches:6MMTACTSMSM
- added S5: CUS-12TB, TiLDA Mk3 Parts:SWITCH-SPST-SMD-A
Connections:
- new net N$3: C42.1, IC8.BAT, JP2.2
- new net N$63: C40.1, IC8.SW, L3.1
- new net N$73: C40.2, IC8.BTST
- new net N$74: C43.1, IC8.REGN, R27.P$1
- new net N$75: C44.1, IC8.PMID
- new net N$76: IC8.!QON, S3.3, S3.4
- new net N$78: IC8.!CE, R23.P$1
- new net N$79: IC8.PSEL, R24.P$1, R25.P$2
- new net N$80: IC8.SCL
- new net N$81: IC8.SDA
- new net N$82: IC8.!INT
- new net N$83: IC8.STAT, R26.P$2
- new net N$84: LED3.C, R26.P$1
- new net N$85: IC8.!PG
- new net N$86: IC8.TS, R27.P$2, R28.P$1
- new net SW: IC9.SW, L4.1
- new net VABT_SWTICHED: Q6.D
- new net VBAT: Q6.S, R45.1
- new net VBAT_SWITCH_CONTROL: Q6.G, R45.2, S5.S
- new net V_UNREG: C41.1, C46.1, IC8.SYS, IC9.EN, IC9.VIN, L3.2, R25.P$1
- net +3V3: now also C45.1, C47.1, IC9.VOS, L4.2
- net GND: now also C39.2, C41.2, C42.2, C43.2, C44.2, C45.2, C46.2, C47.2, IC8.GND, IC9.GND, IC9.MODE, JP2.1, R23.P$2, R24.P$2, R28.P$2, S3.1, S3.2, S5.P
- net USB_VBUS: now also C39.1, IC8.VAC, IC8.VBUS, LED3.A
Other:
- note added: "10V"
- note added: "3V3 Regulator"
- note added: "6mA max"
- note added: "Battery Switch"
- note added: "CONNECT!"
- note added: "POWER SWITCH"
- note added: "SPEC!"

Commit message: connecting some serial interfaces
Connections:
- removed net N$25: IC4.UART1_TX
- removed net N$26: IC4.UART1_RX
- removed net N$46: IC3.UART1_TXD
- removed net N$47: IC3.UART1_RXD
- removed net N$50: IC4.SPI_CLK
- removed net N$51: IC4.SPI_DIN
- removed net N$52: IC4.SPI_DOUT
- removed net N$53: IC4.!SPI_CS
- removed net N$64: J3.SDO
- removed net N$65: J3.SDI
- new net CC_CLK: IC1D.PD3, IC4.SPI_CLK
- new net CC_CS: IC1D.PD2, IC4.!SPI_CS
- new net CC_MISO: IC1D.PD0, IC4.SPI_DOUT
- new net CC_MOSI: IC1D.PD1, IC4.SPI_DIN
- new net CC_RX: IC1D.PD5, IC4.UART1_RX
- new net CC_TX: IC1D.PD4, IC4.UART1_TX
- new net LCD_CLK: IC1A.PA2
- new net LCD_CS: IC1A.PA3
- new net LCD_MISO: IC1A.PA5, J3.SDO
- new net LCD_MOSI: IC1A.PA4, J3.SDI
- new net N$72: IC1K.PK0
- new net SIM_RX: IC1GHJ.PJ1, IC3.UART1_RXD
- new net SIM_TX: IC1GHJ.PJ0, IC3.UART1_TXD
- net S0: now also IC1GHJ.PH0
- net S1: now also IC1GHJ.PH1
- net S2: now also IC1GHJ.PH2
- net S29: now also IC1P.PP2
- net S3: now also IC1GHJ.PH3
- net S30: now also IC1P.PP3
Other:
- note added: "CHECK ALL SPI PINS (TI names are different to mosi etc)"
- note added: "NEEDS LEVEL SHIFTERS!!"
- note removed: "s0, 1, 2, 3, 29, 30"
- note removed: "still to connect:"

Commit message: some more connections done
Parts:
- added C48: 10p, passives-7351:CAPACITOR0603-N
- added C49: 33p, passives-7351:CAPACITOR0603-N
- added C50: 4.7u, passives-7351:CAPACITOR0603-N
- added C51: 100u, TiLDA Mk4 Parts:C-EUC1210
- added LED4: red, TiLDA Mk4 Parts:LED0603
- added Q2, Q3, Q4: (no value), TiLDA Mk4 Parts:MOSFET-N-SOT23-SPARK
- added R29: 10k, passives-7351:RESISTOR0603-N
- added R30: 2k, passives-7351:RESISTOR0603-N
- added S4: (no value), Switches:6MMTACTSMSM
- added U$1: MIC9.7MM, SparkFun-Sensors:MIC9.7MM
Connections:
- removed net N$66: J3.CSX
- new net N$25: IC3.NETLIGHT, Q4.G, R29.P$2
- new net N$26: J3.WRX(D/CX)
- new net N$46: LED4.C, Q4.D
- new net N$52: Q2.G
- new net N$53: IC3.PWRKEY, Q3.D, S4.3, S4.4
- new net N$64: LED4.A, R30.P$1
- new net N$65: Q3.G
- net +3V3: now also R30.P$2
- net GND: now also C48.1, C49.1, C50.1, C51.2, Q2.S, Q3.S, Q4.S, R29.P$1, S4.1, S4.2
- net LCD_CLK: now also J3.D/CX(SCL)
- net LCD_CS: now also J3.CSX
- net N$45: now also C48.2, C49.2, C50.2, C51.1
- net N$60: now also Q2.D
Other:
- note added: "2396073"
- note added: "2724398"
- note added: "MSP423 min hi level: 0.65*3.3 = 2.15V"
- note added: "SIM800C Hi level: 2.4V min"
- note added: "connect"
- note added: "connect?"
- note added: "or tant"
- note removed: "NEEDS LEVEL SHIFTERS!!"

Commit message: adding magjack
Parts:
- added JP3, JP4, JP5: (no value), TiLDA Mk4 Parts:M02PTH
- J1: value MAGJACK -> MAGJACK-RJMG16XXX-8; device SparkFun-Connectors:MAGJACK -> TiLDA Mk4 Parts:MAGJACK-RJMG16XXX-8
Connections:
- net +3V3: now also JP3.1, JP3.2
- net N$20: now also J1.RX-; no longer J1.RD-
- net N$21: now also J1.RX+; no longer J1.RD+
- net N$22: now also J1.TX-; no longer J1.TD-
- net N$23: now also J1.TX+; no longer J1.TD+
- net N$24: now also J1.SHIELD; no longer J1.SHIELD@0, J1.SHIELD@1
- net V_UNREG: now also JP4.1, JP5.1
Other:
- note removed: "CONNECTED CORRECTLY?"
- note removed: "SPEC THIS PART!!!"
- moved on the sheet: C21, C22, C23, R9

Commit message: all major connections done
Parts:
- removed IC4: CC3100MOD-LWK, TiLDA Mk4 Parts:CC3100MOD-LWK
- added C52, C53, C54: 10p, passives-7351:CAPACITOR0603-N
- added C55, C56, C57: 33p, passives-7351:CAPACITOR0603-N
- added IC10: CC3120MOD, TiLDA Mk4 Parts:CC3120MOD
- added LED5: red, TiLDA Mk4 Parts:LED0603
- added R31, R32, R33: dnp, passives-7351:RESISTOR0603-N
- added R34: 2k, passives-7351:RESISTOR0603-N
- added S6: (no value), Switches:6MMTACTSMSM
- R14: value 10k -> 470
- R15: value 220k -> 100k
- R16: value 220k -> 470
Connections:
- removed net N$43: IC3.MICN
- removed net N$44: IC3.MICP
- removed net N$49: IC4.!HIB
- removed net N$52: Q2.G
- removed net N$54: IC4.IRQ
- removed net N$55: IC3.STATUS
- removed net N$61: J3.RESET
- removed net N$65: Q3.G
- removed net N$69: R22.P$2
- removed net N$70: R21.P$2
- removed net N$71: D1.DIN
- removed net N$72: IC1K.PK0
- removed net N$80: IC8.SCL
- removed net N$81: IC8.SDA
- removed net N$82: IC8.!INT
- removed net VABT_SWTICHED: Q6.D
- removed net VBAT: Q6.S, R45.1
- new net BQ_INT: IC1E.PE5, IC8.!INT
- new net BQ_SCL: IC1B.PB4, IC8.SCL
- new net BQ_SDA: IC1B.PB5, IC8.SDA
- new net CC_HIB: IC10.!HIB, IC1E.PE1, R15.P$1
- new net CC_IRQ: IC10.IRQ, IC1E.PE0
- new net CC_RST: IC10.!RESET, IC1K.PK0, S6.3, S6.4
- new net ETHLED0: IC1K.PK4, R14.P$1
- new net ETHLED1: IC1K.PK6, R16.P$1
- new net ETHLED2: IC1F.PF1, R34.P$2
- new net LCD_BLIGHT: IC1F.PF0, Q2.G
- new net LCD_DCX: IC1K.PK2, J3.WRX(D/CX)
- new net LCD_RST: IC1K.PK3, J3.RESET
- new net LCD_TEAR: IC1K.PK1, J3.TE
- new net LEDA: IC1B.PB0, R21.P$2
- new net LEDB: IC1B.PB1, R22.P$2
- new net N$50: C31.1, C32.1, IC10.VBAT_1, IC10.VBAT_2, IC10.VBAT_RESET, JP3.2, R32.P$1
- new net NETLIGHT: IC1P.PP4, IC3.NETLIGHT, Q4.G, R29.P$2
- new net NPIX: D1.DIN, IC1E.PE4
- new net PWR_KEY: IC1Q.PQ4, Q3.G
- new net SIM_STATUS: IC1P.PP5, IC3.STATUS
- new net VBAT_SWITCHED: C46.1, IC9.EN, IC9.VIN, JP4.1, Q6.D, R31.P$2
- new net VBAT_UNSWITCH: JP5.2, Q6.S, R33.P$1, R45.1
- net +3V3: now also J3.RD, JP1.VCC, R32.P$2; no longer C31.1, C32.1, IC4.VBAT_DCDC_ANA, IC4.VBAT_DCDC_DIG, IC4.VBAT_DCDC_PA, JP3.2
- net CC_CLK: now also IC10.SPI_CLK; no longer IC4.SPI_CLK
- net CC_CS: now also IC10.!SPI_CS; no longer IC4.!SPI_CS
- net CC_MISO: now also IC10.SPI_DOUT; no longer IC4.SPI_DOUT
- net CC_MOSI: now also IC10.SPI_DIN; no longer IC4.SPI_DIN
- net CC_RX: now also IC10.UART1_RX; no longer IC4.UART1_RX
- net CC_TX: now also IC10.UART1_TX; no longer IC4.UART1_TX
- net GND: now also C52.2, C54.1, C55.2, C57.1, IC10.GND, J1.LED1-, J1.LED2-, LED5.C, S6.1, S6.2; no longer IC4.GND, R14.P$2, R16.P$2
- net N$25: now also J1.LED1+, R14.P$2; no longer IC3.NETLIGHT, Q4.G, R29.P$2
- net N$26: now also J1.LED2+, R16.P$2; no longer J3.WRX(D/CX)
- net N$36: now also IC1F.PF2; no longer IC4.SOP2, R14.P$1
- net N$37: now also IC1F.PF3; no longer IC4.RESERVED, R15.P$1
- net N$38: now also C52.1, C53.2, C55.1, C56.2, IC3.MICP, U$1.1; no longer IC4.FORCE_AP, R16.P$1
- net N$39: now also LED5.A, R34.P$1; no longer IC4.!RESET
- net N$42: now also C53.1, C54.2, C56.1, C57.2, IC3.MICN, U$1.2; no longer IC6.IO3, U1.USBID
- net N$45: now also JP4.2, R31.P$1
- net N$48: now also IC10.RF_BG; no longer IC4.RF_BG
- net V_UNREG: now also R33.P$2; no longer C46.1, IC9.EN, IC9.VIN, JP4.1
Other:
- note added: "Note: the BQ25601 max sys voltage is very close to the SIM800C Vcc_max"
- note added: "pwm"
- note removed: "??"
- note removed: "CONNECT!"
- note removed: "ESD!"
- moved on the sheet: JP3, JP4, R14, R15, R16, U$1

Commit message: testpoints added
Parts:
- added JP10, JP8: (no value), TiLDA Mk4 Parts:M04PTH
- added JP11, JP13, JP14: (no value), TiLDA Mk4 Parts:M03PTH
- added JP12, JP9: (no value), TiLDA Mk4 Parts:M05PTH
- added JP6, JP7: (no value), TiLDA Mk4 Parts:M07
Connections:
- new net N$43: IC10.TEST_58, JP10.1
- new net N$44: IC10.!UART_RTS, JP9.3
- new net N$49: IC10.!UART_CTS, JP9.2
- new net N$51: IC10.TEST_59, JP10.2
- new net N$52: IC10.TEST_60, JP10.3
- new net N$54: IC10.TEST_62, JP10.4
- new net N$55: IC10.SOP0, JP11.1
- new net N$61: IC10.SOP1, JP11.2
- new net N$65: IC10.SOP2, JP11.3
- new net N$66: IC10.!FLASH_CS, JP12.2
- new net N$69: IC10.FLASH_CLK, JP12.3
- new net N$70: IC10.FLASH_MOSI, JP12.4
- new net N$71: IC10.FLASH_MISO, JP12.5
- new net N$72: IC3.UART2_RXD, JP14.2
- new net N$77: IC3.UART2_TXD, JP14.3
- net BQ_INT: now also JP8.2
- net BQ_SCL: now also JP8.4
- net BQ_SDA: now also JP8.3
- net CC_CLK: now also JP7.6
- net CC_CS: now also JP7.3
- net CC_HIB: now also JP7.7
- net CC_IRQ: now also JP7.2
- net CC_MISO: now also JP7.4
- net CC_MOSI: now also JP7.5
- net CC_RX: now also JP9.4
- net CC_TX: now also JP9.5
- net GND: now also JP12.1, JP13.1, JP14.1, JP6.1, JP7.1, JP8.1, JP9.1
- net LCD_CLK: now also JP6.7
- net LCD_CS: now also JP6.6
- net LCD_DCX: now also JP6.2
- net LCD_MISO: now also JP6.4
- net LCD_MOSI: now also JP6.5
- net LCD_TEAR: now also JP6.3
- net SIM_RX: now also JP13.2
- net SIM_TX: now also JP13.3
Other:
- note removed: "connect"
- note removed: "spi here"

Commit message: a few single testpoints
Parts:
- added TP1, TP2, TP3, TP4, TP5, TP6, TP7, TP8: TP, Testpoint:TP
Connections:
- new net N$80: IC1MISC./HIB, TP7.P$1
- net +3V3: now also TP8.P$1
- net CC_RST: now also TP2.P$1
- net N$40: now also TP5.P$1
- net N$41: now also TP6.P$1
- net N$79: now also TP1.P$1
- net NETLIGHT: now also TP4.P$1
- net SIM_STATUS: now also TP3.P$1
Changed lines of the file:
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@@
 <part name="GND78" library="supply1" deviceset="GND" device=""/>
 <part name="GND79" library="supply1" deviceset="GND" device=""/>
+<part name="TP1" library="Testpoint" deviceset="TP" device=""/>
+<part name="TP2" library="Testpoint" deviceset="TP" device=""/>
+<part name="TP3" library="Testpoint" deviceset="TP" device=""/>
+<part name="TP4" library="Testpoint" deviceset="TP" device=""/>
+<part name="TP5" library="Testpoint" deviceset="TP" device=""/>
+<part name="TP6" library="Testpoint" deviceset="TP" device=""/>
+<part name="TP7" library="Testpoint" deviceset="TP" device=""/>
+<part name="TP8" library="Testpoint" deviceset="TP" device=""/>
 </parts>
 <sheets>
@@
 <instance part="GND78" gate="1" x="99.06" y="-73.66"/>
 <instance part="GND79" gate="1" x="78.74" y="-68.58"/>
+<instance part="TP1" gate="G$1" x="-403.86" y="-68.58"/>
+<instance part="TP2" gate="G$1" x="93.98" y="-195.58"/>
+<instance part="TP3" gate="G$1" x="86.36" y="-40.64" rot="R180"/>
+<instance part="TP4" gate="G$1" x="76.2" y="-17.78"/>
+<instance part="TP5" gate="G$1" x="251.46" y="-27.94"/>
+<instance part="TP6" gate="G$1" x="251.46" y="-30.48" rot="R180"/>
+<instance part="TP7" gate="G$1" x="-198.12" y="104.14" rot="R90"/>
+<instance part="TP8" gate="G$1" x="-134.62" y="294.64" rot="R180"/>
 </instances>
 <busses>
@@
 <junction x="-134.62" y="297.18"/>
 <junction x="-134.62" y="294.64"/>
+<pinref part="TP8" gate="G$1" pin="P$1"/>
 </segment>
 <segment>
@@
 <wire x1="220.98" y1="-27.94" x2="226.06" y2="-27.94" width="0.1524" layer="91"/>
 <junction x="226.06" y="-27.94"/>
-<wire x1="226.06" y1="-27.94" x2="256.54" y2="-27.94" width="0.1524" layer="91"/>
+<wire x1="226.06" y1="-27.94" x2="251.46" y2="-27.94" width="0.1524" layer="91"/>
+<pinref part="TP5" gate="G$1" pin="P$1"/>
+<wire x1="251.46" y1="-27.94" x2="256.54" y2="-27.94" width="0.1524" layer="91"/>
+<junction x="251.46" y="-27.94"/>
 </segment>
 </net>
@@
 <junction x="220.98" y="-35.56"/>
 <wire x1="220.98" y1="-35.56" x2="215.9" y2="-35.56" width="0.1524" layer="91"/>
-<wire x1="256.54" y1="-30.48" x2="233.68" y2="-30.48" width="0.1524" layer="91"/>
+<wire x1="256.54" y1="-30.48" x2="251.46" y2="-30.48" width="0.1524" layer="91"/>
+<wire x1="251.46" y1="-30.48" x2="233.68" y2="-30.48" width="0.1524" layer="91"/>
 <wire x1="233.68" y1="-30.48" x2="233.68" y2="-35.56" width="0.1524" layer="91"/>
 <wire x1="233.68" y1="-35.56" x2="226.06" y2="-35.56" width="0.1524" layer="91"/>
+<pinref part="TP6" gate="G$1" pin="P$1"/>
+<junction x="251.46" y="-30.48"/>
 </segment>
 </net>
@@
 <wire x1="-347.98" y1="-63.5" x2="-360.68" y2="-63.5" width="0.1524" layer="91"/>
 <wire x1="-360.68" y1="-63.5" x2="-360.68" y2="-68.58" width="0.1524" layer="91"/>
-<wire x1="-360.68" y1="-68.58" x2="-408.94" y2="-68.58" width="0.1524" layer="91"/>
+<wire x1="-360.68" y1="-68.58" x2="-403.86" y2="-68.58" width="0.1524" layer="91"/>
 <pinref part="R24" gate="G$1" pin="P$1"/>
+<wire x1="-403.86" y1="-68.58" x2="-408.94" y2="-68.58" width="0.1524" layer="91"/>
 <wire x1="-408.94" y1="-68.58" x2="-411.48" y2="-68.58" width="0.1524" layer="91"/>
 <junction x="-408.94" y="-68.58"/>
 <pinref part="R25" gate="G$1" pin="P$2"/>
+<pinref part="TP1" gate="G$1" pin="P$1"/>
+<junction x="-403.86" y="-68.58"/>
 </segment>
 </net>
@@
 <junction x="71.12" y="-17.78"/>
 <label x="22.86" y="-27.94" size="1.778" layer="95"/>
+<pinref part="TP4" gate="G$1" pin="P$1"/>
 </segment>
 <segment>
@@
 <junction x="93.98" y="-195.58"/>
 <label x="83.82" y="-195.58" size="1.778" layer="95"/>
+<pinref part="TP2" gate="G$1" pin="P$1"/>
 </segment>
 <segment>
@@
 <segment>
 <pinref part="IC3" gate="G$1" pin="STATUS"/>
-<wire x1="99.06" y1="-40.64" x2="78.74" y2="-40.64" width="0.1524" layer="91"/>
+<wire x1="99.06" y1="-40.64" x2="86.36" y2="-40.64" width="0.1524" layer="91"/>
 <label x="78.74" y="-40.64" size="1.778" layer="95"/>
+<pinref part="TP3" gate="G$1" pin="P$1"/>
+<wire x1="86.36" y1="-40.64" x2="78.74" y2="-40.64" width="0.1524" layer="91"/>
+<junction x="86.36" y="-40.64"/>
 </segment>
 </net>
@@
 </segment>
 </net>
+<net name="N$80" class="0">
+<segment>
+<pinref part="IC1" gate="MISC" pin="/HIB"/>
+<pinref part="TP7" gate="G$1" pin="P$1"/>
+</segment>
+</net>

Commit message: ready to start routing
Parts:
- added JP15: JOYSTICK_MINI_MULTICOM_NOSILK, TiLDA Mk4 Parts:JOYSTICK_MINI_MULTICOM_NOSILK
- added R35, R36, R37, R38, R39, R41: 1k, passives-7351:RESISTOR0603-N
- added R40, R42, R43, R44: 5.6k, passives-7351:RESISTOR0603-N
- added TP10, TP11, TP12, TP13, TP9: TP, Testpoint:TP
Connections:
- new net GGGG: IC3.UART1_RXD, R41.P$1, R42.P$1
- new net N$82: IC3.STATUS, R36.P$1
- new net N$91: IC3.UART1_TXD, R37.P$1
- new net N$92: IC3.UART2_RXD, R39.P$1, R40.P$1
- new net N$93: JP14.2, R39.P$2
- new net N$94: IC3.UART1_RTS, TP9.P$1
- new net N$95: IC3.UART1_CTS, TP10.P$1
- new net N$96: IC3.UART1_DCD, TP11.P$1
- new net N$97: IC3.UART1_RI, TP12.P$1
- new net N$98: IC3.UART1_DTR, TP13.P$1
- new net NETLIGHT_: IC3.NETLIGHT, Q4.G, R29.P$2, R35.P$1, TP4.P$1
- net +3V3: now also R43.P$1, R44.P$1
- net BQ_SCL: now also R43.P$2
- net BQ_SDA: now also R44.P$2
- net GND: now also R40.P$2, R42.P$2
- net N$72: now also IC3.UART2_TXD, R38.P$1; no longer IC3.UART2_RXD, JP14.2
- net N$77: now also R38.P$2; no longer IC3.UART2_TXD
- net NETLIGHT: now also R35.P$2; no longer IC3.NETLIGHT, Q4.G, R29.P$2, TP4.P$1
- net SIM_RX: now also R41.P$2; no longer IC3.UART1_RXD
- net SIM_STATUS: now also R36.P$2; no longer IC3.STATUS
- net SIM_TX: now also R37.P$2; no longer IC3.UART1_TXD
Other:
- note removed: "connect?"
- moved on the sheet: ANT1, ANT2, C14, C15, C16, C17, C18, C19, C20, C24, C25, C26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
