File: dev-board1/dev-board1.brd (EAGLE design)
At the start: 100 x 100 mm, 193 parts, among them IC1 MSP432E401, IC10 CC3120MOD, IC11 4066D, IC2 MT48LC16M16A2, IC3 SIM800C, IC4 OPAMP-DUALU, IC5 TPD3E001DRL, IC6 TPD3E001DRL, IC7 TPD3E001DRL, IC8 BQ25601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

Commit message: finishing touches...
Parts:
- R45: value 0603/220k/5% -> 10k; device TiLDA Mk3 Parts:C0603K-SMALL -> passives-7351:R0603-N
- moved JP2 8.29 mm to (3.37, -8.33), turned to 90 degrees
- moved S5 7.14 mm to (12.8, -17.8)
- moved R45 5.98 mm to (12.6, -10.6), turned to 180 degrees
- moved R24 5.89 mm to (8.74, 11.4)
- moved R25 5.89 mm to (7.11, 11.4)
- moved R26 5.89 mm to (10.8, 11.4)
- moved TP1 5.89 mm to (6.50, 9.06)
- moved C39 5.89 mm to (7.72, 7.43)
- moved C40 5.89 mm to (11.8, 1.95)
- moved C43 5.89 mm to (11.8, 3.57)
- moved C44 5.89 mm to (10.4, 6.42)
- moved IC8 5.89 mm to (5.89, 2.56)
- moved L3 5.89 mm to (11.4, -1.51)
- moved LED3 5.89 mm to (12.5, 11.5)
- moved C41 5.89 mm to (7.52, -1.92)
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Connections:
- net GND: now also IC8.25
- net VBAT_SWITCH_CONTROL: now also R45.1; no longer R45.2
- net VBAT_UNSWITCH: now also R45.2; no longer R45.1
Routing:
- net GND: track 468.0 -> 482.4 mm, vias 153 -> 200
- net PWM: track 104.2 -> 95.8 mm, vias 5 -> 4
- net N$76: track 62.5 -> 55.1 mm, vias 2 -> 6
- net +3V3: track 698.8 -> 692.1 mm, vias 39 -> 41
- net VBAT_SWITCHED: track 84.4 -> 78.5 mm
- net N$48: track 9.66 -> 15.1 mm
- net V_UNREG: track 61.8 -> 66.5 mm
- net VBAT_SWITCH_CONTROL: track 12.1 -> 15.3 mm
- net N$3: track 9.15 -> 12.0 mm
- net USB_VBUS: track 130.1 -> 132.7 mm
- net BQ_INT: track 91.1 -> 89.1 mm
- net SSI3FSS: track 24.7 -> 23.0 mm
- net NETLIGHT_: track 47.9 -> 46.3 mm
- net N$62: track 27.5 -> 29.1 mm
- net BQ_SCL: track 98.6 -> 100.0 mm
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Other:
- outline, holes or cut-outs redrawn
- board text added: "1"
- board text added: "2"
- board text added: "58"
- board text added: "59"
- board text added: "60"
- board text added: "62"
- board text added: "A"
- board text added: "April 18"
- board text added: "B"
- board text added: "CC FLASH SPI"
- board text added: "CC PWR"
- board text added: "CC RST"
- board text added: "CTS"
- board text added: "DCD"
- board text added: "DTR"
- board text added: "M. Brejza"
- board text added: "NETLIGHT"
- board text added: "PWM"
- board text added: "QON"
- board text added: "RI"
- board text added: "RST"
- board text added: "RTS"
- board text added: "Rev 1"
- board text added: "S/N:"
- board text added: "SIM PWR"
- board text added: "SOP0"
- board text added: "SOP1"
- board text added: "SOP2"
- board text added: "STATUS"
- board text added: "UART"
- board text added: "WAKE"

Commit message: some tweaks
Parts:
- moved S5 4.51 mm to (8.33, -18.4)
- moved ANT1 3.25 mm to (31.8, -18.6)
Routing:
- net VBAT_SWITCH_CONTROL: track 15.3 -> 20.9 mm
- net N$48: track 15.1 -> 12.7 mm
Other:
- outline, holes or cut-outs redrawn

Commit message: silk tweaks
Parts:
- moved TP2 2.48 mm to (58.1, -17.2)
- moved TP3 2.07 mm to (35.6, 60.4)
Routing:
- net BQ_INT: track 89.1 -> 90.4 mm
- net SIM_STATUS: track 18.7 -> 19.9 mm
- net GND: track 482.7 -> 481.9 mm, vias 200 -> 202
- net SWDAT: track 36.0 -> 36.8 mm
- net N$9: track 37.2 -> 36.6 mm
Other:
- board text added: "Charge"
- board text added: "Status"

Commit message: final prototype 1 (hopefully)
Parts:
- removed TP5, TP6: TP, Testpoint:TP
- added JP18: (no value), TiLDA Mk4 Parts:1X02
- added TP14: TP, Testpoint:TP
Connections:
- net ADC: now also TP14.P$1
- net N$40: now also JP18.1; no longer TP5.P$1
- net N$41: now also JP18.2; no longer TP6.P$1
Routing:
- net GND: track 481.9 -> 467.7 mm, vias 202 -> 217
- net ADC: track 35.0 -> 36.9 mm
- net N$41: track 30.9 -> 32.1 mm
- net N$40: track 37.5 -> 36.8 mm, vias 4 -> 3
- net N$9: track 36.6 -> 36.0 mm
Other:
- board text added: "ADC"
- board text added: "SPEAKER"

Commit message: adding part numbers
Parts:
- R43, R44: value 5.6k -> 4.7k

Commit message: adding final few farnell numbers
Parts:
- L3: value (none) -> 1.5u
Changed lines of the file:
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@@
 <attribute name="NAME" x="24.277378125" y="39.1286" size="0.8128" layer="25" font="vector" ratio="13"/>
 </element>
-<element name="ANT1" library="TiLDA Mk4 Parts" package="2450AT42A100" value="CHIPANT" x="31.75" y="-18.6284" smashed="yes" rot="R180"/>
+<element name="ANT1" library="TiLDA Mk4 Parts" package="2450AT42A100" value="CHIPANT" x="31.75" y="-18.6284" smashed="yes" rot="R180">
+<attribute name="FARNELL" value="2148522" x="31.75" y="-18.6284" size="1.778" layer="27" rot="R180" display="off"/>
+</element>
 <element name="C31" library="TiLDA Mk4 Parts" package="C1210" value="100u" x="59.69" y="-11.9228" smashed="yes" rot="R90">
 <attribute name="FARNELL" value="1889302" x="59.69" y="-11.9228" size="1.778" layer="27" rot="R90" display="off"/>
@@
 </element>
 <element name="C34" library="passives-7351" package="C0603-N" value="4.7u" x="92.6084" y="26.4132" smashed="yes">
+<attribute name="FARNELL" value="2524873" x="92.6084" y="26.4132" size="1.778" layer="27" display="off"/>
 <attribute name="NAME" x="94.3616" y="26.0068" size="0.8128" layer="25" font="vector" ratio="13"/>
 </element>
@@
 </element>
 <element name="X2" library="con-coax" package="BU-SMA-V" value="BU-SMA-V" x="10.3632" y="75.3872" smashed="yes" rot="MR0">
+<attribute name="FARNELL" value="1248990" x="10.3632" y="75.3872" size="1.778" layer="28" rot="MR0" display="off"/>
 <attribute name="MF" value="" x="10.3632" y="75.3872" size="1.778" layer="28" rot="MR0" display="off"/>
 <attribute name="MPN" value="" x="10.3632" y="75.3872" size="1.778" layer="28" rot="MR0" display="off"/>
@@
 <attribute name="OC_NEWARK" value="unknown" x="10.3632" y="75.3872" size="1.778" layer="28" rot="MR0" display="off"/>
 </element>
-<element name="ANT2" library="TiLDA Mk4 Parts" package="2450AT42A100" value="CHIPANT" x="36.576" y="78.6384" smashed="yes"/>
-<element name="J4" library="dtb" package="SWD_PTH_SHROUD" value="SWD_SHROUD" x="39.4208" y="66.4464" smashed="yes"/>
+<element name="ANT2" library="TiLDA Mk4 Parts" package="2450AT42A100" value="CHIPANT" x="36.576" y="78.6384" smashed="yes">
+<attribute name="FARNELL" value="2148522" x="36.576" y="78.6384" size="1.778" layer="27" display="off"/>
+</element>
+<element name="J4" library="dtb" package="SWD_PTH_SHROUD" value="SWD_SHROUD" x="39.4208" y="66.4464" smashed="yes">
+<attribute name="FARNELL" value="1865285" x="39.4208" y="66.4464" size="1.778" layer="27" display="off"/>
+</element>
 <element name="JP1" library="tag-connect" package="TC2030-MCP-NL" value="TC2030-SWDNL" x="45.5168" y="67.8688" smashed="yes" rot="MR90"/>
 <element name="IC8" library="TiLDA Mk4 Parts" package="QFN-24" value="BQ25601" x="5.8928" y="2.5552" smashed="yes" rot="R270"/>
@@
 </element>
 <element name="JP2" library="TiLDA Mk4 Parts" package="JST-2-SMD" value="" x="3.368" y="-8.3312" smashed="yes" rot="R90">
+<attribute name="FARNELL" value="9492615" x="3.368" y="-8.3312" size="1.778" layer="27" rot="R90" display="off"/>
 <attribute name="NAME" x="4.056028125" y="-13.6742" size="0.8128" layer="25" font="vector" ratio="14"/>
 <attribute name="VALUE" x="3.368" y="-9.6012" size="0.4064" layer="27" rot="R90"/>
 </element>
-<element name="L3" library="TiLDA Mk4 Parts" package="1008" value="" x="11.3792" y="-1.5088" smashed="yes" rot="R270">
+<element name="L3" library="TiLDA Mk4 Parts" package="1008" value="1.5u" x="11.3792" y="-1.5088" smashed="yes" rot="R270">
 <attribute name="FARNELL" value="2428202" x="11.3792" y="-1.5088" size="1.778" layer="27" rot="R270" display="off"/>
 <attribute name="NAME" x="13.6264" y="-1.6096" size="0.8128" layer="25" font="vector" ratio="14" rot="R90"/>
@@
 </element>
 <element name="C41" library="passives-7351" package="C0805-N" value="10u" x="7.5184" y="-1.9152" smashed="yes">
+<attribute name="FARNELL" value="2112853/2362101/2576756" x="7.5184" y="-1.9152" size="1.778" layer="27" display="off"/>
 <attribute name="NAME" x="7.01588125" y="-3.940525" size="0.8128" layer="25" font="vector" ratio="13"/>
 </element>
 <element name="C43" library="passives-7351" package="C0603-N" value="4.7u" x="11.7856" y="3.5712" smashed="yes">
+<attribute name="FARNELL" value="2524873" x="11.7856" y="3.5712" size="1.778" layer="27" display="off"/>
 <attribute name="NAME" x="13.5388" y="3.1648" size="0.8128" layer="25" font="vector" ratio="13"/>
 </element>
 <element name="C44" library="passives-7351" package="C0805-N" value="10u" x="10.3632" y="6.416" smashed="yes" rot="R90">
+<attribute name="FARNELL" value="2112853/2362101/2576756" x="10.3632" y="6.416" size="1.778" layer="27" rot="R90" display="off"/>
 <attribute name="NAME" x="11.572221875" y="9.1018" size="0.8128" layer="25" font="vector" ratio="13" rot="R180"/>
 </element>
 <element name="C42" library="passives-7351" package="C0805-N" value="10u" x="3.2512" y="-1.9152" smashed="yes" rot="R180">
+<attribute name="FARNELL" value="2112853/2362101/2576756" x="3.2512" y="-1.9152" size="1.778" layer="27" rot="R180" display="off"/>
 <attribute name="NAME" x="4.97291875" y="-3.141075" size="0.8128" layer="25" font="vector" ratio="13" rot="R180"/>
 </element>
@@
 </element>
 <element name="C45" library="TiLDA Mk3 Parts" package="C0805-N" value="0805/10u/10V/X5R" x="20.9296" y="0.9296" smashed="yes">
+<attribute name="FARNELL" value="2112853/2362101/2576756" x="20.9296" y="0.9296" size="1.778" layer="27" display="off"/>
 <attribute name="NAME" x="19.3838" y="1.3056" size="0.8128" layer="25" font="vector" ratio="13" rot="R180"/>
 </element>
 <element name="C46" library="TiLDA Mk3 Parts" package="C0805-N" value="0805/10u/10V/X5R" x="20.9296" y="-6.792" smashed="yes">
+<attribute name="FARNELL" value="2112853/2362101/2576756" x="20.9296" y="-6.792" size="1.778" layer="27" display="off"/>
 <attribute name="NAME" x="19.8338" y="-8.6208" size="0.8128" layer="25" font="vector" ratio="13"/>
 </element>
@@
 </element>
 <element name="C47" library="TiLDA Mk3 Parts" package="C0805-N" value="0805/10u/10V/X5R" x="20.9296" y="-1.1024" smashed="yes">
+<attribute name="FARNELL" value="2112853/2362101/2576756" x="20.9296" y="-1.1024" size="1.778" layer="27" display="off"/>
 <attribute name="NAME" x="19.3838" y="0.0864" size="0.8128" layer="25" font="vector" ratio="13" rot="R180"/>
 </element>
@@
 </element>
 <element name="C50" library="passives-7351" package="C0603-N" value="4.7u" x="1.6256" y="67.4624" smashed="yes" rot="R270">
+<attribute name="FARNELL" value="2524873" x="1.6256" y="67.4624" size="1.778" layer="27" rot="R270" display="off"/>
 <attribute name="NAME" x="2.524678125" y="69.02130625" size="0.8128" layer="25" font="vector" ratio="13" rot="R270"/>
 </element>
@@
 <element name="TP12" library="Testpoint" package="TP" value="TP" x="16.0528" y="55.0672" smashed="yes" rot="R90"/>
 <element name="TP13" library="Testpoint" package="TP" value="TP" x="14.4272" y="55.0672" smashed="yes" rot="R90"/>
-<element name="JP15" library="TiLDA Mk4 Parts" package="JOYSTICK_MULTICOMP_NOSILK" value="JOYSTICK_MINI_MULTICOM_NOSILK" x="49.9872" y="49.1744" smashed="yes" rot="MR45"/>
+<element name="JP15" library="TiLDA Mk4 Parts" package="JOYSTICK_MULTICOMP_NOSILK" value="JOYSTICK_MINI_MULTICOM_NOSILK" x="49.9872" y="49.1744" smashed="yes" rot="MR45">
+<attribute name="FARNELL" value="1316987" x="49.9872" y="49.1744" size="1.778" layer="28" rot="MR45" display="off"/>
+</element>
 <element name="R43" library="passives-7351" package="R0603-N" value="4.7k" x="13.208" y="7.0256" smashed="yes" rot="R270">
 <attribute name="NAME" x="14.137721875" y="8.68749375" size="0.8128" layer="25" font="vector" ratio="13" rot="R90"/>
@@
 </element>
 <element name="IC4" library="SparkFun-AnalogIC" package="SO08" value="OPAMP-DUALU" x="28.0416" y="24.9936" smashed="yes">
+<attribute name="FARNELL" value="2463666" x="28.0416" y="24.9936" size="1.778" layer="27" display="off"/>
 <attribute name="NAME" x="31.4196" y="24.12751875" size="0.8128" layer="25" font="vector" ratio="13" rot="R90"/>
 </element>
