File: Mk4 Prototype.sch (EAGLE design)
At the start: 6 parts

Commit message: Initial shape and some layout ideas
Parts:
- added ARTWORK1: ARTWORK_JOYSTICK, TiLDA Mk4 Parts:ARTWORK_JOYSTICK
- added ARTWORK2: ARTWORK_KEYPAD, TiLDA Mk4 Parts:ARTWORK_KEYPAD
- added C1: 0603 1u/10V/X5R, TiLDA Mk4 Parts:C-EUC0603K-SMALL
- added C38: 0603 4u7/10V/X5R, TiLDA Mk4 Parts:C-EUC0603K-SMALL
- added C45: 0603 100n/10V/X5R, TiLDA Mk4 Parts:C-EUC0603K-SMALL
- added IC1: MSP432E401, TiLDA Mk4 Parts:MSP432E401
- added IC2: AS4C8M16SA-7TCN, TiLDA Mk4 Parts:MT48LCXXM16A2TG
- added IC3: CC3120MOD, TiLDA Mk4 Parts:CC3120MOD
- added IC5: SIM800C, TiLDA Mk4 Parts:SIM800C
- added J2: ER-CON50HT-1, TiLDA Mk4 Parts:ER-TFT024-3
- added J3: 2x5 1.27mm (NP), TiLDA Mk4 Parts:SWD_SHROUD-PINHEAD
- added JP1: (no value), TiLDA Mk4 Parts:M02-JST-2MM-SMT
- added JP2: 1x03, TiLDA Mk4 Parts:M03LOCK
- added JP4: (NP), TiLDA Mk4 Parts:TC2030-SWDNL
- added LAYERS1: LAYER_NUMBRS_4_SMALL, TiLDA Mk4 Parts:LAYER_NUMBRS_4_SMALL
- added LED1, LED2: (no value), TiLDA Mk4 Parts:WS2812B
- added OUTLINE1: TILDA_MK3_BOARDOUTLINE-MK4, TiLDA Mk4 Parts:TILDA_MK3_BOARDOUTLINE-MK4
- added Q8: CSD13202Q2, TiLDA Mk4 Parts:CSD13202Q2
- added R44, R47, R48, R49: 0603 12R/5%, TiLDA Mk4 Parts:R-EU_0603K-SMALL
- added S1, S10, S11, S12, S13, S14, S15, S2, S3, S4, S5, S6, S7, S8, S9: SKPMAPE010, TiLDA Mk4 Parts:TAC_SWITCH1-SKPMAPE010
- added S16, S17: 3X6X2.5, TiLDA Mk4 Parts:TAC_SWITCH1-3X6X2.5
- added S18: CUS-12TB, TiLDA Mk4 Parts:SWITCH-SPST-SMD-A
- added SW1: JOYSTICK, TiLDA Mk4 Parts:JOYSTICK_MINI_MULTICOM_NOSILK
- added TP1, TP2, TP21, TP3, TP4: (NP), TiLDA Mk4 Parts:TPB1,27
- added U2: ER-TFT024-3 (NP), TiLDA Mk4 Parts:ER-TFT024-3-OUTLINE
- FID1, FID2, FID3, FID4, FID5, FID6: device TiLDA Mk3 Parts:FIDUCIAL1X2.5-STOP -> TiLDA Mk4 Parts:FIDUCIAL1X2.5-STOP
Connections:
- new net 3V3: C38.2, C45.2, IC2_PWR.VDD, IC2_PWR.VDDQ, J2.LEDA, J2.VCI, J2.VDDI, J3.VCC, JP4.VCC, OUTLINE1.3V3, SW1.COM
- new net ADC_X: J2.X-
- new net ADC_Y: J2.Y-
- new net BTN_1: S1.3
- new net BTN_10: S10.3
- new net BTN_11: S11.3
- new net BTN_12: S12.3
- new net BTN_2: S2.3
- new net BTN_3: S3.3
- new net BTN_4: S4.3
- new net BTN_5: S5.3
- new net BTN_6: S6.3
- new net BTN_7: S7.3
- new net BTN_8: S8.3
- new net BTN_9: S9.3
- new net BTN_A: S13.3
- new net BTN_B: S15.3
- new net BTN_CALL: S16.3
- new net BTN_END: S17.3
- new net BTN_MENU: S14.3
- new net FSMC_A23: J2.D/CX(SCL), TP4.TP
- new net GND: C1.2, C38.1, C45.1, IC2_PWR.VSS, IC2_PWR.VSSQ, J2.DB10, J2.DB11, J2.DB12, J2.DB13, J2.DB14, J2.DB15, J2.DB16, J2.DB17, J2.DB8, J2.DB9, J2.DE, J2.DOTCLK, J2.GND, J2.HSYNC, J2.IM0, J2.VSYNC, J3.GND1, J3.GND2, J3.GNDD, JP1.1, JP2.1, JP4.GND, LED1.VSS, LED2.VSS, OUTLINE1.GND, Q8.S, S1.1, S10.1, S11.1, S12.1, S13.1, S14.1, S15.1, S16.1, S17.1, S2.1, S3.1, S4.1, S5.1, S6.1, S7.1, S8.1, S9.1
- new net JOY_CEN: SW1.CENT
- new net JOY_DOWN: SW1.DOWN
- new net JOY_LEFT: SW1.LEFT
- new net JOY_RIGHT: SW1.RIGHT
- new net JOY_UP: SW1.UP
- new net LCD0: J2.DB0, TP1.TP
- new net LCD1: J2.DB1
- new net LCD2: J2.DB2
- new net LCD3: J2.DB3
- new net LCD4: J2.DB4
- new net LCD5: J2.DB5
- new net LCD6: J2.DB6
- new net LCD7: J2.DB7
- new net LCD_!RST: J2.RESET
- new net LCD_CS: J2.CSX
- new net LCD_MODE: J2.IM1, J2.IM2, J2.IM3
- new net LCD_RD: J2.RD, TP2.TP
- new net LCD_WRX: J2.WRX(D/CX), TP3.TP
- new net LEDK1: J2.LEDK1, R47.2
- new net LEDK2: J2.LEDK2, R48.2
- new net LEDK3: J2.LEDK3, R49.2
- new net LEDK4: J2.LEDK4, R44.2
- new net N$64: Q8.D, R44.1, R47.1, R48.1, R49.1
- new net NRST: J3.NRST, JP4.RST
- new net PA0: IC1_A.PA0
- new net PA1: IC1_A.PA1
- new net PA2: IC1_A.PA2
- new net PA3: IC1_A.PA3
- new net PA4: IC1_A.PA4
- new net PA5: IC1_A.PA5
- new net PB0: IC1_B.PB0
- new net PB1: IC1_B.PB1
- new net PB2: IC1_B.PB2
- new net PB4: IC1_B.PB4
- new net PB5: IC1_B.PB5
- new net PD0: IC1_D.PD0
- new net PD1: IC1_D.PD1
- new net PD2: IC1_D.PD2
- new net PD3: IC1_D.PD3
- new net PD4: IC1_D.PD4
- new net PD5: IC1_D.PD5
- new net PD6: IC1_D.PD6
- new net PD7: IC1_D.PD7
- new net PE0: IC1_E.PE0
- new net PE1: IC1_E.PE1
- new net PE2: IC1_E.PE2
- new net PE3: IC1_E.PE3
- new net PE4: IC1_E.PE4
- new net PE5: IC1_E.PE5
- new net PF0: IC1_F.PF0
- new net PF1: IC1_F.PF1
- new net PF2: IC1_F.PF2
- new net PF3: IC1_F.PF3
- new net PF4: IC1_F.PF4
- new net PJ0: IC1_GHJ.PJ0
- new net PJ1: IC1_GHJ.PJ1
- new net PK0: IC1_K.PK0
- new net PK1: IC1_K.PK1
- new net PK2: IC1_K.PK2
- new net PK3: IC1_K.PK3
- new net PK4: IC1_K.PK4
- new net PK6: IC1_K.PK6
- new net PK7: IC1_K.PK7
- new net PL4: IC1_L.PL4
- new net PL5: IC1_L.PL5
- new net PM4: IC1_M.PM4
- new net PM5: IC1_M.PM5
- new net PM6: IC1_M.PM6
- new net PM7: IC1_M.PM7
- new net PN0: IC1_N.PN0
- new net PN1: IC1_N.PN1
- new net PN2: IC1_N.PN2
- new net PN3: IC1_N.PN3
- new net PN4: IC1_N.PN4
- new net PN5: IC1_N.PN5
- new net PP0: IC1_P.PP0
- new net PP1: IC1_P.PP1
- new net PP4: IC1_P.PP4
- new net PP5: IC1_P.PP5
- new net PQ0: IC1_Q.PQ0
- new net PQ1: IC1_Q.PQ1
- new net PQ2: IC1_Q.PQ2
- new net PQ3: IC1_Q.PQ3
- new net PQ4: IC1_Q.PQ4
- new net SDRAM_!CAS: IC1_L.PL2, IC2G$1.!CAS
- new net SDRAM_!CS: IC1_P.PP2, IC2G$1.\CS
- new net SDRAM_!RAS: IC1_L.PL3, IC2G$1.!RAS
- new net SDRAM_!WE: IC1_B.PB3, IC2G$1.!WE
- new net SDRAM_A0: IC1_GHJ.PH0, IC2G$1.A0, IC2G$1.DQ0
- new net SDRAM_A1: IC1_GHJ.PH1, IC2G$1.A1, IC2G$1.DQ1
- new net SDRAM_A10: IC1_GHJ.PG1, IC2G$1.A10, IC2G$1.DQ10
- new net SDRAM_A11: IC1_GHJ.PG0, IC2G$1.A11, IC2G$1.DQ11
- new net SDRAM_A12: IC1_M.PM3, IC2G$1.A12, IC2G$1.DQ12
- new net SDRAM_A2: IC1_GHJ.PH2, IC2G$1.A2, IC2G$1.DQ2
- new net SDRAM_A3: IC1_GHJ.PH3, IC2G$1.A3, IC2G$1.DQ3
- new net SDRAM_A4: IC1_C.PC7, IC2G$1.A4, IC2G$1.DQ4
- new net SDRAM_A5: IC1_C.PC6, IC2G$1.A5, IC2G$1.DQ5
- new net SDRAM_A6: IC1_C.PC5, IC2G$1.A6, IC2G$1.DQ6
- new net SDRAM_A7: IC1_C.PC4, IC2G$1.A7, IC2G$1.DQ7
- new net SDRAM_A8: IC1_A.PA6, IC2G$1.A8, IC2G$1.DQ8
- new net SDRAM_A9: IC1_A.PA7, IC2G$1.A9, IC2G$1.DQ9
- new net SDRAM_BA0: IC1_M.PM2, IC2G$1.BA0, IC2G$1.DQ13
- new net SDRAM_BA1: IC1_M.PM1, IC2G$1.BA1, IC2G$1.DQ14
- new net SDRAM_CKE: IC1_P.PP3, IC2G$1.CKE
- new net SDRAM_CLK: IC1_K.PK5, IC2G$1.CLK
- new net SDRAM_D15: IC1_M.PM0, IC2G$1.DQ15
- new net SDRAM_DQMH: IC1_L.PL1, IC2G$1.DQMH
- new net SDRAM_DQML: IC1_L.PL0, IC2G$1.DQML
- new net SPI3_MISO: J2.SDO
- new net SPI3_MOSI: J2.SDI
- new net TCK_SWCLK: IC1_C.PC0, J3.SWCLK, JP4.SWCLK
- new net TDI: IC1_C.PC2
- new net TDO_SWO: IC1_C.PC3
- new net TEAR: J2.TE, TP21.TP
- new net TIM17_CH1: Q8.G
- new net TMS_SWDIO: IC1_C.PC1, J3.SWDAT, JP4.SWDAT
- new net T_X: J2.X+
- new net T_Y: J2.Y+
- new net USB_D_N: IC1_L.PL7
- new net USB_D_P: IC1_L.PL6
- new net VBAT: JP1.2
- new net V_UNREG: C1.1, JP2.2, LED1.VDD, LED2.VDD
- new net WS2812: LED1.DIN
- new net WS2812_OUT: JP2.3, LED2.DOUT
- new net WS28212_1: LED1.DOUT, LED2.DIN
Other:
- note added: "+"
- note added: "-"
- note added: "Battery Connection"
- note added: "Front Buttons"
- note added: "JTAG"
- note added: "JTAG SWD"
- note added: "LCD Screen"
- note added: "LCD_MODE 0: parallel; 1: serial"
- note added: "NC in 128M"
- note added: "POE Wurth Socket 7499210001A"

Commit message: Drop in a few more parts and identified some options for Spk, MIC and antennas
Parts:
- added IC4: MCP23017ML, TiLDA Mk4 Parts:MCP23017ML
- added IC6: SST26VF064B-104I/SM, TiLDA Mk4 Parts:SPI_FLASH-X25XXSMD1
- added J1: 78723-1001, TiLDA Mk4 Parts:SIM-78723-1001-LWK
- added J4: ANTENNA-GSM, TiLDA Mk4 Parts:ANTENNA-GSM
- added JP3: 1x11, TiLDA Mk4 Parts:M11LOCK
- added JP5, JP6: 1x08, TiLDA Mk4 Parts:M08LOCK
- added U1: (no value), TiLDA Mk4 Parts:USB-AB-LWK
Connections:
- new net BT_ANT: IC5.BT_ANT
- new net GSM_ANT: IC5.GSM_ANT, J4.1
- new net N$36: IC3.RF_BG
- net TDI: now also J3.NC
- net TDO_SWO: now also J3.SWO, JP4.SWO
- net V_UNREG: now also OUTLINE1.VBATT
Other:
- note added: "2450AT18D0100"
- note added: "CMA-4544PF-W"
- note added: "CMC-6022-37T"
- note added: "CMS-15118D-SP"
- note added: "ETH"
- note added: "GPIO0"
- note added: "GPIO1"
- note added: "MO044402-10"
- note added: "Mic"
- note added: "Outline Conductive Pads"
- note added: "Spk"
- moved on the sheet: IC2

Commit message: NIght 2
Parts:
- removed JP3: 1x11, TiLDA Mk4 Parts:M11LOCK
- removed TP2, TP21, TP3, TP4: (NP), TiLDA Mk4 Parts:TPB1,27
- added C10, C11, C12, C13, C15, C2, C21, C22, C23, C24, C25, C26, C27, C28, C3, C4, C5, C8, C9: 0402/100n/10V/X5R, TiLDA Mk4 Parts:C-EUC0402-SMALLER
- added C14, C7: 0603/1u/10V/X5R, TiLDA Mk4 Parts:C-EUC0603K-SMALL
- added C16, C17, C18, C19: 0402/12p/50V/C0G, TiLDA Mk4 Parts:C-EUC0402-SMALLER
- added C20: 0603/3300p/50V/X7R, TiLDA Mk4 Parts:C-EUC0603K-SMALL
- added C6: 0603/2u2/10V/X5R, TiLDA Mk4 Parts:C-EUC0603K-SMALL
- added IC7: TPD3E001DRL, TiLDA Mk4 Parts:TPD3E001DRL
- added JP7: 1x14, TiLDA Mk4 Parts:M14LOCK
- added L2: BLM18KG121TN1D, TiLDA Mk4 Parts:WE-CBF_0805
- added LED3: 0603 RED, TiLDA Mk4 Parts:LED0603-CORRECT
- added LED4: 0603 GREEN, TiLDA Mk4 Parts:LED0603-CORRECT
- added LED5: (no value), TiLDA Mk4 Parts:LED5MM
- added Q3: CSD13202Q2, TiLDA Mk3 Parts:CSD13202Q2
- added R1, R2: 0402/1K/5%, TiLDA Mk4 Parts:R-EU_R0402-SMALLER
- added R10, R9: 0402/10k/5%, TiLDA Mk4 Parts:R-EU_R0402-SMALLER
- added R11: (no value), TiLDA Mk4 Parts:R-EU_0309/10
- added R12: 0402/2k/5%, TiLDA Mk4 Parts:R-EU_R0402-SMALLER
- added R14: 0402/4k7/5%, TiLDA Mk4 Parts:R-EU_R0402-SMALLER
- added R3: 0402/4k87/5%, TiLDA Mk4 Parts:R-EU_R0402-SMALLER
- added R4: 0402/10K/5%, TiLDA Mk4 Parts:R-EU_R0402-SMALLER
- added R5, R7: 0402/1M/5%, TiLDA Mk4 Parts:R-EU_R0402-SMALLER
- added R6: 0402/2K/5%, TiLDA Mk4 Parts:R-EU_R0402-SMALLER
- added R8: 0402/100/5%, TiLDA Mk4 Parts:R-EU_R0402-SMALLER
- added S19, S20: 3X6X2.5, TiLDA Mk4 Parts:TAC_SWITCH1-3X6X2.5
- added X1: FC-135R 32.768KHZ 9PF, TiLDA Mk4 Parts:RESONATOR_EPSON_FC_145
- added X2: NX3225GA-25.000M-STD-CRG-2, TiLDA Mk4 Parts:CRYSTAL-3.2-2.5
- C1: value 0603 1u/10V/X5R -> 0603/1u/10V/X5R
- C38: value 0603 4u7/10V/X5R -> 0603/4u7/10V/X5R
- C45: value 0603 100n/10V/X5R -> 0402/100n/10V/X5R; device TiLDA Mk4 Parts:C-EUC0603K-SMALL -> TiLDA Mk4 Parts:C-EUC0402-SMALLER
- R44, R47, R48, R49: value 0603 12R/5% -> 0402/12R/5%; device TiLDA Mk4 Parts:R-EU_0603K-SMALL -> TiLDA Mk4 Parts:R-EU_R0402-SMALLER
- TP1: value (NP) -> TP; TP_SIGNAL_NAME (none) -> !HIB
Connections:
- net PP1 renamed SSI3DAT3
- removed net FSMC_A23: J2.D/CX(SCL), TP4.TP
- removed net LCD0: J2.DB0, TP1.TP
- removed net LCD1: J2.DB1
- removed net LCD2: J2.DB2
- removed net LCD3: J2.DB3
- removed net LCD4: J2.DB4
- removed net LCD5: J2.DB5
- removed net LCD6: J2.DB6
- removed net LCD7: J2.DB7
- removed net LCD_MODE: J2.IM1, J2.IM2, J2.IM3
- removed net LCD_RD: J2.RD, TP2.TP
- removed net LCD_WRX: J2.WRX(D/CX), TP3.TP
- removed net PA2: IC1_A.PA2
- removed net PA3: IC1_A.PA3
- removed net PA4: IC1_A.PA4
- removed net PA5: IC1_A.PA5
- removed net PB0: IC1_B.PB0
- removed net PB1: IC1_B.PB1
- removed net PF0: IC1_F.PF0
- removed net PF4: IC1_F.PF4
- removed net PK1: IC1_K.PK1
- removed net PK2: IC1_K.PK2
- removed net PK3: IC1_K.PK3
- removed net PK4: IC1_K.PK4
- removed net PK6: IC1_K.PK6
- removed net PM4: IC1_M.PM4
- removed net PM5: IC1_M.PM5
- removed net PM7: IC1_M.PM7
- removed net PN0: IC1_N.PN0
- removed net PP0: IC1_P.PP0
- removed net PQ0: IC1_Q.PQ0
- removed net PQ1: IC1_Q.PQ1
- removed net PQ2: IC1_Q.PQ2
- removed net PQ3: IC1_Q.PQ3
- removed net SPI3_MISO: J2.SDO
- removed net SPI3_MOSI: J2.SDI
- removed net TEAR: J2.TE, TP21.TP
- removed net TIM17_CH1: Q8.G
- new net !CC_HIB: IC3.!HIB
- new net !CC_RST: IC3.!RESET
- new net !HIB: IC1_MISC./HIB, TP1.TP
- new net !RESET: C15.2, IC1_MISC./RST, J3.NRST, R4.1, S19.3
- new net !WAKE: IC1_MISC./WAKE, R5.1, S20.3
- new net 3V3_POE: C5.2, JP7.14
- new net CC_IRQ: IC3.IRQ
- new net CH1: OUTLINE1.CH1
- new net CH2: OUTLINE1.CH2
- new net CH3: OUTLINE1.CH3
- new net CH4: OUTLINE1.CH4
- new net EN0RXI_N: IC1_MISC.EN0RXIN, JP7.13
- new net EN0RXI_P: IC1_MISC.EN0RXIP, JP7.11
- new net EN0TXO_N: IC1_MISC.EN0TXON, JP7.7
- new net EN0TXO_P: IC1_MISC.EN0TXOP, JP7.6
- new net ETHLED0: IC1_K.PK4, R1.2
- new net ETHLED1: IC1_K.PK6, R2.2
- new net FET: Q3.G
- new net FET_OUT: LED5.C, OUTLINE1.FET, Q3.D
- new net I2C2_SCL: OUTLINE1.SCL
- new net I2C2_SDA: OUTLINE1.SDA
- new net I2C_SCL: IC4.SCL
- new net I2C_SDA: IC4.SDA
- new net LCD_BLIGHT: IC1_F.PF0, Q8.G
- new net LCD_CLK: IC1_A.PA2, J2.D/CX(SCL)
- new net LCD_DCX: IC1_K.PK2, J2.WRX(D/CX)
- new net LCD_MISO: IC1_A.PA5, J2.SDO
- new net LCD_MOSI: IC1_A.PA4, J2.SDI
- new net LCD_TEAR: IC1_K.PK1, J2.TE
- new net LED1: IC1_B.PB0, R12.2
- new net LED2: IC1_B.PB1, R14.2
- new net MCP_INT: IC4.INTA
- new net N$1: LED5.A, R11.1
- new net N$3: JP7.3, R1.1
- new net N$4: JP7.5, R2.1
- new net N$5: IC1_MISC.RBIAS, R3.1
- new net N$51: LED4.A, R14.1
- new net N$52: LED3.A, R12.1
- new net N$6: C20.2, R7.1, U1.SHIELD
- new net OSC0: C16.2, IC1_MISC.OSC0, X2.C1
- new net OSC1: IC1_MISC.OSC1, R6.1
- new net OSC1_R: C17.2, R6.2, X2.C2
- new net SPI1_MISO: IC3.SPI_DOUT
- new net SPI1_MOSI: IC3.SPI_DIN
- new net SPI1_NSS: IC3.!SPI_CS
- new net SPI1_SCK: IC3.SPI_CLK
- new net SSI3_CLK: IC1_Q.PQ0, IC6.SCK
- new net SSI3_DAT0: IC1_Q.PQ2, IC6.MOSI
- new net SSI3_DAT1: IC1_Q.PQ3, IC6.MISO
- new net SSI3_DAT2: IC1_F.PF4, IC6.WP, R10.2
- new net SSI3_DAT3: IC6.HOLD, R9.2
- new net SSI3_FSS: IC1_Q.PQ1, IC6.CS
- new net USART1_RX: IC3.UART1_TX
- new net USART1_TX: IC3.UART1_RX
- new net USB_ID: R8.2
- new net USB_ID_R: IC7.IO3, R8.1, U1.USBID
- new net VBUS: IC7.VCC, L2.2
- new net VBUS_L: L2.1, U1.VBUS
- new net VDDC: C6.2, C7.2, C8.2, IC1_PWR.VDDC
- new net XOSC0: C18.2, IC1_MISC.XOSC0, X1.1
- new net XOSC1: C19.2, IC1_MISC.XOSC1, X1.2
- net 3V3: now also C10.2, C11.2, C12.2, C13.2, C14.2, C2.2, C21.2, C22.2, C23.2, C24.2, C25.2, C26.2, C27.2, C28.2, C3.2, C4.2, C9.2, IC1_PWR.REFA+, IC1_PWR.VBAT, IC1_PWR.VDD, IC1_PWR.VDDA, IC4.VDD, IC6.VCC, J2.IM1, J2.IM2, J2.IM3, J2.RD, JP7.12, JP7.8, R10.1, R11.2, R4.2, R5.2, R9.1
- net BTN_1: now also IC4.GPA0
- net BTN_10: now also IC4.GPB1
- net BTN_11: now also IC4.GPB2
- net BTN_12: now also IC4.GPB3
- net BTN_2: now also IC4.GPA1
- net BTN_3: now also IC4.GPA2
- net BTN_4: now also IC4.GPA3
- net BTN_5: now also IC4.GPA4
- net BTN_6: now also IC4.GPA5
- net BTN_7: now also IC4.GPA6
- net BTN_8: now also IC4.GPA7
- net BTN_9: now also IC4.GPB0
- net BTN_A: now also IC4.GPB6
- net BTN_B: now also IC4.GPB7
- net BTN_CALL: now also IC4.GPB4
- net BTN_END: now also IC4.GPB5
- net GND: now also C10.1, C11.1, C12.1, C13.1, C14.1, C15.1, C16.1, C17.1, C18.1, C19.1, C2.1, C20.1, C21.1, C22.1, C23.1, C24.1, C25.1, C26.1, C27.1, C28.1, C3.1, C4.1, C5.1, C6.1, C7.1, C8.1, C9.1, IC1_PWR.GND, IC1_PWR.GNDA, IC4.A0, IC4.A1, IC4.A2, IC4.VSS, IC6.GND, IC7.GND, J2.DB0, J2.DB1, J2.DB2, J2.DB3, J2.DB4, J2.DB5, J2.DB6, J2.DB7, JP5.1, JP6.1, JP7.1, JP7.2, JP7.4, LED3.C, LED4.C, Q3.S, R3.2, R7.2, S19.1, S20.1, U1.GND, X2.GND@1, X2.GND@2
- net JOY_CEN: now also IC1_P.PP0
- net JOY_DOWN: now also IC1_N.PN0
- net JOY_LEFT: now also IC1_M.PM5
- net JOY_RIGHT: now also IC1_M.PM4
- net JOY_UP: now also IC1_M.PM7
- net LCD_!RST: now also IC1_K.PK3
- net LCD_CS: now also IC1_A.PA3
- net NRST: no longer J3.NRST
- net USB_D_N: now also IC7.IO1, U1.D-
- net USB_D_P: now also IC7.IO2, U1.D+
Other:
- note added: "A"
- note added: "ADC pins for touch?"
- note added: "B"
- note added: "Edge pins"
- note added: "LEDs"
- note added: "Or Ours with POE"
- note added: "SDRAM"
- note added: "SQI FLASH"
- note added: "Spackfun BOB-13021"
- note added: "do we need wake"
- note added: "lcd_blight on PWM?"
- note added: "ws2812 on pwm or timmer?"
- moved on the sheet: IC1_MISC, IC1_PWR, IC4, IC6, JP5, JP6, OUTLINE1, TP1, U1
