File: Mk4 Prototype.brd (EAGLE design)
At the start: 121.6 x 80 mm, 108 parts, among them IC1 MSP432E401, IC2 AS4C8M16SA-7TCN, IC3 CC3120MOD, IC4 MCP23017ML, IC5 SIM800C, IC6 SST26VF064B-104I/SM, IC7 TPD3E001DRL, J1 78723-1001, J2 ER-CON50HT-1, J3 2x5 1.27mm (NP), J4 ANTENNA-GSM, Q3 CSD13202Q2, Q8 CSD13202Q2, SW1 JOYSTICK, U2 ER-TFT024-3 (NP), X1 FC-135R 32.768KHZ 9PF, X2 NX3225GA-25.000M-STD-CRG-2

Commit message: Day 3
Parts:
- added ANT1: 24509AT1BD100, TiLDA Mk4 Parts:2450AT18D0100-RIGHT
- added ANT2: 24509AT1BD100, TiLDA Mk4 Parts:2450AT18D0100
- added C29, C32: 1411/100u/10V/Tant, TiLDA Mk4 Parts:CT3528
- added C30, C39: 0603/4u7/10V/X5R, TiLDA Mk4 Parts:C0603K-SMALL
- added C31, C44, C51, C70, C71: 0402/100n/10V/X5R, TiLDA Mk4 Parts:C0402-SMALLER
- added C33, C34, C35, C36, C40, C46, C47: 0805/10u/10V/X5R, TiLDA Mk4 Parts:C0805-N
- added C37: 0402/??/10V/X5R, TiLDA Mk4 Parts:C0402-SMALLER
- added C41: 0603/1u/10V/X5R, TiLDA Mk4 Parts:C0603K-SMALL
- added C42, C43: 1210/100u/6V3/X5R, TiLDA Mk4 Parts:C1210K
- added C48, C49, C50: 0402/22p/10V/X5R, TiLDA Mk4 Parts:C0402-SMALLER
- added C52, C54, C55, C58, C60, C61, C64, C66, C67: 0402/33p/50V/X5R, TiLDA Mk4 Parts:C0402-SMALLER
- added C53, C56, C57, C59, C62, C63, C65, C68, C69: 0402/10p/50V/X5R, TiLDA Mk4 Parts:C0402-SMALLER
- added C72, C73, C74, C75, C76, C77: (no value), TiLDA Mk4 Parts:C0402-SMALLER
- added D1: MMSZ5231BT1G, TiLDA Mk4 Parts:SOD123
- added D2: LXES15AAA1-153, TiLDA Mk4 Parts:R0402-SMALLER
- added IC10: TPD3E001DRL, TiLDA Mk4 Parts:DRL-5
- added IC11: LMV358ID, TiLDA Mk4 Parts:SO08-SPARK-NEW
- added IC12: SN74HC4066D, TiLDA Mk4 Parts:SO14
- added IC8: BQ25601, TiLDA Mk4 Parts:QFN-24
- added IC9: TPS62082, TiLDA Mk4 Parts:WSON8
- added JP3: 1x02 2MM, TiLDA Mk4 Parts:1X02_2MM
- added JP8, JP9: 1x04_1.27MM, TiLDA Mk4 Parts:1X04-1.27MM
- added L1, L4: SRN2512-2R2M, TiLDA Mk4 Parts:1008
- added L3, L5, L6: 0402/0R/5%, TiLDA Mk4 Parts:L0402
- added LED6: 0603 RED, TiLDA Mk4 Parts:LED-0603-CORRECT
- added Q1, Q2: 2N7002PW, TiLDA Mk4 Parts:SC70-3-R
- added R13, R15, R16, R18, R19, R20: 0402/10k/5%, TiLDA Mk4 Parts:R0402-SMALLER
- added R17: 0402/2k/5%, TiLDA Mk4 Parts:R0402-SMALLER
- added R21, R22, R23, R24: 0402/4k7/5%, TiLDA Mk4 Parts:R0402-SMALLER
- added R25, R30: 0402/100k/5%, TiLDA Mk4 Parts:R0402-SMALLER
- added R26, R27, R28: 0402/51R/5%, TiLDA Mk4 Parts:R0402-SMALLER
- added R29: 0402/4K7/5%, TiLDA Mk4 Parts:R0402-SMALLER
- added R31, R32, R33, R34, R35, R36, R37, R41, R42: 0402/1K/5%, TiLDA Mk4 Parts:R0402-SMALLER
- added R38, R39, R40: 0402/5K6/5%, TiLDA Mk4 Parts:R0402-SMALLER
- added R43, R45, R46: 0402/10K/5%, TiLDA Mk4 Parts:R0402-SMALLER
- added R50, R51: 0402/22K/5%, TiLDA Mk4 Parts:R0402-SMALLER
- added U4: MIC-1X02, TiLDA Mk4 Parts:1X02
- added U5: LDMS1540S-01-R8-0.8-R, TiLDA Mk4 Parts:SPEAKER-15MM-SMD
- J4: value ANTENNA-GSM -> GSM-COIL-ANT
- JP1: value (none) -> S2B-PH-SM4-TB(LF)(SN)
- LED1, LED2: value (none) -> WS2812B
- LED5: value (none) -> LED 5MM
- Q3: value CSD13202Q2 -> CSD25402Q3A; device TiLDA Mk3 Parts:Q2 -> TiLDA Mk4 Parts:Q3A
- moved Q3 8.00 mm to (-20.5, 16.0)
- moved J3 1.50 mm to (29.9, 61.0)
- moved C2 1.27 mm to (10.2, 46.2)
- moved R11 1.00 mm to (-35.0, 13.0)
Connections:
- removed net I2C_SCL: IC4.8
- removed net I2C_SDA: IC4.9
- removed net N$36: IC3.31
- removed net PB4: IC1.121
- removed net PB5: IC1.120
- removed net USB_VBUS: IC5.24
- removed net VBAT_1: IC3.37
- removed net VBAT_2: IC3.40
- removed net VCC: J1.C1
- new net BQ_!CE: IC8.9, R17.1
- new net BQ_!INT: IC8.7
- new net BQ_!PG: IC8.3
- new net BQ_PMID: C36.1, IC8.23
- new net BQ_PSEL: IC8.2, R18.1, R19.1
- new net BQ_REGN: C39.2, IC8.22, R16.2
- new net BQ_STAT: IC8.4, R20.1
- new net BQ_SW: C37.2, IC8.19, IC8.20, L1.1
- new net BQ_TS: IC8.11, R15.2, R16.1
- new net BT_ANT_L: ANT2.1, C75.2, L5.2
- new net FLASH_!CS: IC3.14, JP8.2
- new net FLASH_CLK: IC3.15, JP8.3
- new net FLASH_MISO: IC3.13, JP8.1
- new net FLASH_MOSI: IC3.17, JP8.4
- new net GMS_ANT_L: C73.2, D2.1, J4.ANT, L3.2
- new net I2C5_SCL: IC1.121, IC4.8, IC8.5, R22.1
- new net I2C5_SDA: IC1.120, IC4.9, IC8.6, R21.1
- new net MIC_N: C52.2, C53.1, C55.1, C56.2, IC5.10, U4.2
- new net MIC_P: C52.1, C54.1, C56.1, C57.1, IC5.9, U4.1
- new net N$13: LED6.C, R20.2
- new net N$14: Q3.4, R13.1, S18.3
- new net N$17: C37.1, IC8.21
- new net N$19: IC8.12, JP3.2
- new net NETLIGHT: R42.1
- new net NETLIGHT_R: IC5.41, R42.2
- new net PWR_KEY: Q1.1, R30.1
- new net PWR_KEY_FET: IC5.39, Q1.3
- new net SIM_CLK: IC10.2, J1.C3, R27.2
- new net SIM_CLK_R: C49.2, IC5.16, R27.1
- new net SIM_CTS: R34.1
- new net SIM_CTS_R: IC5.4, R34.2
- new net SIM_DATA: IC10.1, J1.C7, R26.2
- new net SIM_DATA_R: C50.2, IC5.15, R26.1
- new net SIM_DCD: R33.1
- new net SIM_DCD_R: IC5.5, R33.2
- new net SIM_DET: IC5.14, J1.C8, R29.2
- new net SIM_DTR: R31.1
- new net SIM_DTR_R: IC5.6, R31.2, R40.1
- new net SIM_D_N: IC5.26, JP9.2
- new net SIM_D_P: IC5.25, JP9.3
- new net SIM_RI: R32.1
- new net SIM_RI_R: IC5.7, R32.2
- new net SIM_RST: IC10.4, J1.C2, R28.2
- new net SIM_RST_R: C48.2, IC5.17, R28.1
- new net SIM_RTS: R35.1
- new net SIM_RTS_R: IC5.3, R35.2, R39.1
- new net SIM_RXD: R37.1
- new net SIM_RXD_R: IC5.2, R37.2, R38.1
- new net SIM_STATUS: R41.1
- new net SIM_STATUS_R: IC5.42, R41.2
- new net SIM_TXD: R36.1
- new net SIM_TXD_R: IC5.1, R36.2
- new net SIM_VBUS: IC5.24, JP9.4
- new net SPK_ADC: IC11.7, R46.2
- new net SPK_N: C58.2, C59.1, C61.1, C62.2, C64.2, C65.1, C67.1, C68.2, IC5.12, R43.1, U5.-
- new net SPK_P: C58.1, C60.1, C62.1, C63.1, C64.1, C66.1, C68.1, C69.1, IC5.11, R45.1, U5.+
- new net SPK_R_N: IC11.5, R45.2, R46.1
- new net SPK_R_P: IC11.6, R43.2, R50.1, R51.1
- new net SW: IC9.7, L4.1
- new net VBATT: C29.+, C30.2, C31.2, C32.+, C46.1, D1.C, IC5.34, IC5.35, IC9.1, IC9.8, Q3.1, Q3.2, Q3.3
- new net WFIF_ANT_L: ANT1.4, C77.2, L6.2
- new net WIFI_ANT: C76.2, IC3.31, L6.1
- net !CC_HIB: now also R25.1
- net 3V3: now also C33.1, C42.2, C43.2, C44.2, C47.1, C70.2, C71.2, IC11.8, IC12.14, IC3.36, IC3.37, IC3.40, IC9.5, L4.2, R21.2, R22.2, R23.2, R24.2, R50.2
- net BT_ANT: now also C74.2, L5.1
- net FET: now also Q2.1; no longer Q3.3
- net FET_OUT: now also Q2.3; no longer Q3.1, Q3.2, Q3.5, Q3.6, Q3.EP1
- net GND: now also ANT1.1, ANT1.2, ANT1.3, ANT2.2, ANT2.3, ANT2.4, C29.-, C30.1, C31.1, C32.-, C33.2, C34.2, C35.2, C36.2, C39.1, C40.2, C41.2, C42.1, C43.1, C44.1, C46.2, C47.2, C48.1, C49.1, C50.1, C51.1, C53.2, C54.2, C55.2, C57.2, C59.2, C60.2, C61.2, C63.2, C65.2, C66.2, C67.2, C69.2, C70.1, C71.1, C72.1, C73.1, C74.1, C75.1, C76.1, C77.1, D1.A, D2.2, IC10.3, IC11.4, IC12.7, IC8.17, IC8.18, IC8.25, IC9.2, IC9.3, IC9.EP, JP3.1, JP9.1, Q1.2, Q2.2, R15.1, R17.2, R19.2, R25.2, R30.2, R38.2, R39.2, R40.2, R51.2, S18.2; no longer Q3.4, Q3.EP2
- net GSM_ANT: now also C72.2, L3.1; no longer J4.ANT
- net I2C2_SCL: now also R24.1
- net I2C2_SDA: now also R23.1
- net SIM_VDD: now also C51.2, IC10.5, J1.C1
- net VBAT: now also C34.1, C35.1, IC8.13, IC8.14; no longer IC5.34, IC5.35
- net VBUS: now also C41.1, IC8.1, IC8.24, LED6.A
- net VDD_EXT: now also R29.1
- net V_UNREG: now also C40.1, IC8.15, IC8.16, L1.2, Q3.5, Q3.6, Q3.7, Q3.8, Q3.EP, R13.2, R18.2
Routing:
- net GND: track 63.1 -> 72.5 mm, vias 70 -> 102
- net VBAT: track 0.00 -> 7.05 mm, vias 0 -> 4
- net BQ_PSEL: track 0.00 -> 3.55 mm
- net I2C5_SCL: track 0.00 -> 2.51 mm
- net I2C5_SDA: track 0.00 -> 1.80 mm
- net 3V3: vias 32 -> 37

Commit message: Schematic should now have all the parts
Parts:
- removed C59, C62, C63: 0402/10p/50V/X5R, TiLDA Mk4 Parts:C0402-SMALLER
- removed C60, C61: 0402/33p/50V/X5R, TiLDA Mk4 Parts:C0402-SMALLER
- added C78: 0402/1n/10V/X5R, TiLDA Mk4 Parts:C0402-SMALLER
- added C79: 0402/2n2/10V/X5R, TiLDA Mk4 Parts:C0402-SMALLER
- added C80, C81: 0402/100n/10V/X5R, TiLDA Mk4 Parts:C0402-SMALLER
- added C82, C83: 0402/220n/6V/X5R, TiLDA Mk4 Parts:C0402-SMALLER
- added IC13: TPA2066D1, TiLDA Mk4 Parts:VSON-8
- added R52: 0402/14K7/5%, TiLDA Mk4 Parts:R0402-SMALLER
- added R53: 0402/7K87/5%, TiLDA Mk4 Parts:R0402-SMALLER
- added R54, R55, R56: 0402/10K/5%, TiLDA Mk4 Parts:R0402-SMALLER
- added R57, R58: 0402/150K/1%, TiLDA Mk4 Parts:R0402-SMALLER
- added R59: 0402/10k/5%, TiLDA Mk4 Parts:R0402-SMALLER
- added SJ1: (no value), TiLDA Mk4 Parts:SJ_3
- C58: value 0402/33p/50V/X5R -> 0402/100n/10V/X5R
- U4: value MIC-1X02 -> MIC-4MM; device TiLDA Mk4 Parts:1X02 -> TiLDA Mk4 Parts:MIC-SMD-4MM
- moved Q2 81.5 mm to (47.0, 11.0), turned to 90 degrees
- moved C58 4.26 mm to (-37.2, 27.2)
- moved U4 2.12 mm to (42.0, 61.5)
- moved C71 1.00 mm to (35.5, 60.5)
- turned C47 to 0 degrees
- turned C65 to 90 degrees
- turned C67 to 90 degrees
- turned U5 to 90 degrees
Connections:
- new net MIC_MUX_N: IC12.11, IC12.9, IC5.10
- new net MIC_MUX_P: IC12.1, IC12.3, IC5.9
- new net MIC_PWM: R53.2
- new net MIC_PWM_AMP: C79.1, C80.2, C81.2, IC11.1, IC11.2
- new net MIC_PWM_N: C80.1, IC12.8, R54.1
- new net MIC_PWM_P: C81.1, IC12.4, R54.2
- new net MUX_A: IC12.12, IC12.13, R56.1
- new net MUX_B: IC12.5, IC12.6, R55.2
- new net N$10: IC13.4, R58.2
- new net N$11: IC13.3, R57.2
- new net N$12: C83.1, R57.1
- new net N$15: C82.1, R58.1
- new net N$2: C78.2, IC11.3, R52.2
- new net N$7: C79.2, R52.1, R53.1
- new net N$9: C58.1, IC13.1, IC13.6, SJ1.2
- new net SPK_AMP_N: IC13.8, U5.-
- new net SPK_AMP_P: IC13.5, U5.+
- net 3V3: now also R56.2
- net FET: now also R59.1
- net GND: now also C58.2, C78.1, IC13.7, IC13.PAD, R55.1, R59.2; no longer C59.2, C60.2, C61.2, C63.2
- net MIC_N: now also IC12.10, U4.-; no longer IC5.10, U4.2
- net MIC_P: now also IC12.2, U4.+; no longer IC5.9, U4.1
- net SPK_N: now also C82.2; no longer C58.2, C59.1, C61.1, C62.2, U5.-
- net SPK_P: now also C83.2; no longer C58.1, C60.1, C62.1, C63.1, U5.+
- net VBATT: now also C1.1, JP2.2, LED1.1, LED2.1
- net V_UNREG: no longer C1.1, JP2.2, LED1.1, LED2.1
Routing:
- net MIC_MUX_N: track 0.00 -> 16.6 mm
- net MIC_N: track 0.00 -> 8.79 mm
- net MIC_PWM_P: track 0.00 -> 7.78 mm
- net MIC_MUX_P: track 0.00 -> 7.45 mm
- net MIC_P: track 0.00 -> 5.01 mm
- net MIC_PWM_N: track 0.00 -> 3.86 mm
- net GND: vias 102 -> 106
- net 3V3: vias 37 -> 39
Other:
- outline, holes or cut-outs redrawn
- board text removed: "TIM2"

Commit message: WIP
Parts:
- J3: value 2x5 1.27mm (NP) -> 2x5 1.27mm
- JP4: value (NP) -> TC2030-MCP-NL
- SJ1: value (none) -> Amp Power Select
- U1: value (none) -> ZX62-AB-5PA(11)
Connections:
- net N$9 renamed AMP_VDD
- net 3V3: now also SJ1.1
- net VBATT: now also SJ1.3
Routing:
- net 3V3: track 33.1 -> 34.0 mm
Changed lines of the file:
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@@
 <setting verticaltext="up"/>
 </settings>
-<grid distance="1" unitdist="mm" unit="mm" style="lines" multiple="1" display="yes" altdistance="0.5" altunitdist="mm" altunit="mm"/>
+<grid distance="0.5" unitdist="mm" unit="mm" style="lines" multiple="1" display="yes" altdistance="0.25" altunitdist="mm" altunit="mm"/>
 <layers>
 <layer number="1" name="Top" color="4" fill="1" visible="yes" active="yes"/>
@@
 <element name="ARTWORK1" library="TiLDA Mk4 Parts" package="TILDA_ARTWORK_JOYSTICK" value="ARTWORK_JOYSTICK" x="-39.2" y="39" locked="yes"/>
 <element name="ARTWORK2" library="TiLDA Mk4 Parts" package="TILDA_ARTWORK_KEYPAD" value="ARTWORK_KEYPAD" x="0" y="0" locked="yes"/>
-<element name="J3" library="TiLDA Mk4 Parts" package="PINHEAD_2X05_127" value="2x5 1.27mm (NP)" x="29.9" y="60.95" rot="MR0">
+<element name="J3" library="TiLDA Mk4 Parts" package="PINHEAD_2X05_127" value="2x5 1.27mm" x="29.9" y="60.95" rot="MR0">
+<attribute name="DNP" value="Y" x="29.9" y="60.95" size="1.778" layer="28" rot="MR0" display="off"/>
 <attribute name="FARNELL" value="1865285" x="29.9" y="60.95" size="1.778" layer="28" rot="MR0" display="off"/>
 </element>
-<element name="JP4" library="TiLDA Mk4 Parts" package="TC2030-MCP-NL" value="(NP)" x="24.3" y="56.85" rot="MR90"/>
+<element name="JP4" library="TiLDA Mk4 Parts" package="TC2030-MCP-NL" value="TC2030-MCP-NL" x="24.3" y="56.85" rot="MR90">
+<attribute name="DNP" value="Y" x="24.3" y="56.85" size="1.778" layer="28" rot="MR90" display="off"/>
+</element>
 <element name="C1" library="TiLDA Mk4 Parts" package="C0603K-SMALL" value="0603/1u/10V/X5R" x="-7.6" y="75.8" rot="MR270"/>
 <element name="JP2" library="TiLDA Mk4 Parts" package="1X03_LOCK" value="1x03" x="-2.54" y="75.4" locked="yes" rot="MR180">
@@
 <attribute name="DNP" value="Y" x="-18" y="75" size="1.778" layer="28" rot="MR345" display="off"/>
 </element>
-<element name="U1" library="TiLDA Mk4 Parts" package="USB-AB-MICRO-SMD_LWK" value="" x="10.4" y="75.5" rot="MR274"/>
+<element name="U1" library="TiLDA Mk4 Parts" package="USB-AB-MICRO-SMD_LWK" value="ZX62-AB-5PA(11)" x="10.4" y="75.5" rot="MR274"/>
 <element name="J1" library="TiLDA Mk4 Parts" package="MSIM-MOLEX-LWK" value="78723-1001" x="57" y="21" rot="MR180"/>
 <element name="J4" library="TiLDA Mk4 Parts" package="GSM-ANTENNA" value="GSM-COIL-ANT" x="56.5" y="36" rot="MR0"/>
@@
 <element name="C58" library="TiLDA Mk4 Parts" package="C0402-SMALLER" value="0402/100n/10V/X5R" x="-37.25" y="27.25" rot="MR90"/>
 <element name="R59" library="TiLDA Mk4 Parts" package="R0402-SMALLER" value="0402/10k/5%" x="45" y="11" rot="MR90"/>
-<element name="SJ1" library="TiLDA Mk4 Parts" package="SJ_3" value="" x="-34.5" y="31" rot="MR0"/>
+<element name="SJ1" library="TiLDA Mk4 Parts" package="SJ_3" value="Amp Power Select" x="-34.5" y="31" rot="MR0">
+<attribute name="DNP" value="Y" x="-34.5" y="31" size="1.778" layer="28" rot="MR0" display="off"/>
+</element>
 </elements>
 <signals>
@@
 <via x="-30.5" y="25" extent="1-16" drill="0.3"/>
 <via x="-29.75" y="25" extent="1-16" drill="0.3"/>
-<via x="-32" y="28.25" extent="1-16" drill="0.3"/>
+<via x="-32.5" y="31" extent="1-16" drill="0.3"/>
 <via x="-37.5" y="37.25" extent="1-16" drill="0.3"/>
+<contactref element="SJ1" pad="1"/>
+<wire x1="-33.611" y1="31" x2="-34.5" y2="31" width="0.15" layer="16"/>
 <wire x1="35" y1="61.5" x2="35" y2="60.5" width="0" layer="19" extent="16-16"/>
 <wire x1="18" y1="49.75" x2="18" y2="49" width="0" layer="19" extent="16-16"/>
@@
 <wire x1="-56" y1="18.25" x2="-57.623" y2="19.56" width="0" layer="19" extent="16-16"/>
 <wire x1="-27.75" y1="20.85" x2="-30.3" y2="20" width="0" layer="19" extent="16-16"/>
+<wire x1="-33.611" y1="31" x2="-32.5" y2="31" width="0" layer="19" extent="16-16"/>
 <wire x1="-2" y1="56.5" x2="-4.75" y2="59.5" width="0" layer="19" extent="16-16"/>
 <wire x1="-2" y1="55.5" x2="-2" y2="56.5" width="0" layer="19" extent="16-16"/>
@@
 <contactref element="C1" pad="1"/>
 <contactref element="JP2" pad="2"/>
+<contactref element="SJ1" pad="3"/>
 <wire x1="0" y1="75.527" x2="5.05" y2="75.6" width="0" layer="19" extent="1-1"/>
 <wire x1="-7.6" y1="76.675" x2="0" y2="75.527" width="0" layer="19" extent="16-16"/>
 <wire x1="-9.95" y1="75.6" x2="-7.6" y2="76.675" width="0" layer="19" extent="1-16"/>
-<wire x1="34.25" y1="25.5" x2="5.05" y2="75.6" width="0" layer="19" extent="1-16"/>
+<wire x1="-35.389" y1="31" x2="-9.95" y2="75.6" width="0" layer="19" extent="1-16"/>
+<wire x1="-32.2" y1="18.5" x2="-35.389" y2="31" width="0" layer="19" extent="16-16"/>
+<wire x1="-30.3" y1="18.5" x2="-32.2" y2="18.5" width="0" layer="19" extent="16-16"/>
+<wire x1="-30.35" y1="16.75" x2="-30.3" y2="18.5" width="0" layer="19" extent="16-16"/>
+<wire x1="-20.825" y1="14.45" x2="-30.35" y2="16.75" width="0" layer="19" extent="16-16"/>
+<wire x1="-20.175" y1="14.45" x2="-20.825" y2="14.45" width="0" layer="19" extent="16-16"/>
+<wire x1="-19.525" y1="14.45" x2="-20.175" y2="14.45" width="0" layer="19" extent="16-16"/>
+<wire x1="34.25" y1="25.5" x2="-19.525" y2="14.45" width="0" layer="19" extent="16-16"/>
 <wire x1="38" y1="25.5" x2="34.25" y2="25.5" width="0" layer="19" extent="16-16"/>
 <wire x1="40.75" y1="25.1" x2="38" y2="25.5" width="0" layer="19" extent="16-16"/>
@@
 <wire x1="43.8" y1="32.2" x2="43.75" y2="30.5" width="0" layer="19" extent="16-16"/>
 <wire x1="44.9" y1="32.2" x2="43.8" y2="32.2" width="0" layer="19" extent="16-16"/>
-<wire x1="-19.525" y1="14.45" x2="34.25" y2="25.5" width="0" layer="19" extent="16-16"/>
-<wire x1="-20.175" y1="14.45" x2="-19.525" y2="14.45" width="0" layer="19" extent="16-16"/>
-<wire x1="-20.825" y1="14.45" x2="-20.175" y2="14.45" width="0" layer="19" extent="16-16"/>
-<wire x1="-30.35" y1="16.75" x2="-20.825" y2="14.45" width="0" layer="19" extent="16-16"/>
-<wire x1="-30.3" y1="18.5" x2="-30.35" y2="16.75" width="0" layer="19" extent="16-16"/>
-<wire x1="-32.2" y1="18.5" x2="-30.3" y2="18.5" width="0" layer="19" extent="16-16"/>
 </signal>
 <signal name="WIFI_ANT" class="1">
@@
 <wire x1="-35.975" y1="28.225" x2="-50.75" y2="30" width="0" layer="19" extent="16-16"/>
 </signal>
-<signal name="N$9">
+<signal name="AMP_VDD">
 <contactref element="IC13" pad="1"/>
 <contactref element="IC13" pad="6"/>

Commit message: Tweaks for BOM
Parts:
- C37: value 0402/??/10V/X5R -> 0402/47n/10V/X5R
- R10, R13, R15, R16, R18, R19, R20, R59, R9: value 0402/10k/5% -> 0402/10K/5%
- R12, R17: value 0402/2k/5% -> 0402/2K/5%
- R14, R21, R22, R23, R24: value 0402/4k7/5% -> 0402/4K7/5%
- R25, R30: value 0402/100k/5% -> 0402/100K/5%
- R3: value 0402/4k87/5% -> 0402/4K87/5%
- R8: value 0402/100/5% -> 0402/100R/5%
- U2: value ER-TFT024-3 (NP) -> ER-TFT024-3
