File: Mk4 Prototype.brd (EAGLE design)
At the start: 121.6 x 80 mm, 222 parts, among them IC1 MSP432E401, IC10 TPD3E001DRL, IC11 LMV358ID, IC12 SN74HC4066D, IC13 TPA2066D1, IC2 AS4C8M16SA-7TCN, IC3 CC3120MOD, IC4 MCP23017ML, IC5 SIM800C, IC6 SST26VF064B-104I/SM, IC7 TPD3E001DRL, IC8 BQ25601, IC9 TPS62082, J1 78723-1001, J2 ER-CON50HT-1, J3 2x5 1.27mm, J4 GSM-COIL-ANT, Q1 2N7002PW, Q2 2N7002PW, Q3 CSD25402Q3A, Q8 CSD13202Q2, SW1 JOYSTICK, U1 ZX62-AB-5PA(11), U2 ER-TFT024-3, U4 MIC-4MM, U5 LDMS1540S-01-R8-0.8-R, X1 FC-135R 32.768KHZ 9PF, X2 NX3225GA-25.000M-STD-CRG-2

Commit message: Tweaks for BOM 2
Parts:
- added BATT: 1000mAh JST-PH, TiLDA Mk4 Parts:BATTERY-32X50
- ANT1, ANT2: value 24509AT1BD100 -> 2450AT18D0100
- IC13: value TPA2066D1 -> TPA2006D1
- IC2: value AS4C8M16SA-7TCN -> AS4C4M16SA-7TCN
- IC6: value SST26VF064B-104I/SM -> SST26VF016B-104I/SM
- PCB: value TILDA_MK3_BOARDOUTLINE-MK4 -> TiLDA Mk4 PCB
- U1: value ZX62-AB-5PA(11) -> ZX62-B-5PA(33)
- X1: value FC-135R 32.768KHZ 9PF -> ABS07-32.768KHZ-T
- X2: value NX3225GA-25.000M-STD-CRG-2 -> ABM8G-25.000MHZ-B4Y-T
- renumbered JP1 to J5, OUTLINE1 to PCB, U2 to LCD
Changed lines of the file:
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@@
 <attribute name="DNP" value="Y" x="-62" y="28" size="1.778" layer="27" rot="R180" display="off"/>
 </element>
-<element name="OUTLINE1" library="TiLDA Mk4 Parts" package="TILDA_MK4_OUTLINE" value="TILDA_MK3_BOARDOUTLINE-MK4" x="0" y="0" locked="yes">
-<attribute name="DNP" value="Y" x="0" y="0" size="1.778" layer="27" display="off"/>
-</element>
+<element name="PCB" library="TiLDA Mk4 Parts" package="TILDA_MK4_OUTLINE" value="TiLDA Mk4 PCB" x="0" y="0" locked="yes"/>
 <element name="IC3" library="TiLDA Mk4 Parts" package="CC3100MOD-LWK" value="CC3120MOD" x="-44.925" y="49.9" rot="MR0"/>
 <element name="R47" library="TiLDA Mk4 Parts" package="R0402-SMALLER" value="0402/12R/5%" x="12.5" y="39" rot="MR270"/>
@@
 <element name="Q8" library="TiLDA Mk4 Parts" package="Q2" value="CSD13202Q2" x="14.5" y="38.75" rot="MR270"/>
 <element name="C45" library="TiLDA Mk4 Parts" package="C0402-SMALLER" value="0402/100n/10V/X5R" x="-8.25" y="39" rot="MR180"/>
-<element name="U2" library="TiLDA Mk4 Parts" package="ER-TFT024-3" value="ER-TFT024-3" x="0" y="33.5" locked="yes" smashed="yes">
-<attribute name="DNP" value="Y" x="0" y="33.5" size="1.778" layer="27" display="off"/>
-</element>
+<element name="LCD" library="TiLDA Mk4 Parts" package="ER-TFT024-3" value="ER-TFT024-3" x="0" y="33.5" locked="yes" smashed="yes"/>
 <element name="SW1" library="TiLDA Mk4 Parts" package="JOYSTICK_MULTICOMP_NOSILK" value="JOYSTICK" x="-39.2" y="39" locked="yes" smashed="yes" rot="R315">
 <attribute name="VALUE" x="-35.3109125" y="40.76776875" size="0.4064" layer="27" rot="R315"/>
@@
 <attribute name="VALUE" x="11.5" y="72.4" size="0.6096" layer="27"/>
 </element>
-<element name="IC2" library="TiLDA Mk4 Parts" package="TSOP54-400" value="AS4C8M16SA-7TCN" x="-21.8" y="52.7" rot="MR270"/>
+<element name="IC2" library="TiLDA Mk4 Parts" package="TSOP54-400" value="AS4C4M16SA-7TCN" x="-21.8" y="52.7" rot="MR270"/>
 <element name="S16" library="TiLDA Mk4 Parts" package="TACTILE_SWITCH_SMD_3X6X2.5H" value="3X6X2.5" x="-30" y="68" locked="yes" smashed="yes" rot="R15">
 <attribute name="VALUE" x="-32.4906" y="66.0903125" size="0.8128" layer="27" rot="R15"/>
@@
 </element>
 <element name="IC1" library="TiLDA Mk4 Parts" package="QFP128-0.4" value="MSP432E401" x="0" y="53" rot="MR0"/>
-<element name="JP1" library="TiLDA Mk4 Parts" package="JST-2-SMD" value="S2B-PH-SM4-TB(LF)(SN)" x="28.8" y="15.8" rot="MR90"/>
+<element name="J5" library="TiLDA Mk4 Parts" package="JST-2-SMD" value="S2B-PH-SM4-TB(LF)(SN)" x="28.8" y="15.8" rot="MR90"/>
 <element name="IC5" library="TiLDA Mk4 Parts" package="SIM800C" value="SIM800C" x="40.5" y="41" rot="MR180"/>
 <element name="ARTWORK1" library="TiLDA Mk4 Parts" package="TILDA_ARTWORK_JOYSTICK" value="ARTWORK_JOYSTICK" x="-39.2" y="39" locked="yes">
@@
 </element>
 <element name="IC4" library="TiLDA Mk4 Parts" package="QFN28-ML_6X6MM" value="MCP23017ML" x="17.5" y="27" rot="MR0"/>
-<element name="IC6" library="TiLDA Mk4 Parts" package="SO08-EIAJ" value="SST26VF064B-104I/SM" x="13.2" y="43.15" rot="MR270"/>
+<element name="IC6" library="TiLDA Mk4 Parts" package="SO08-EIAJ" value="SST26VF016B-104I/SM" x="13.2" y="43.15" rot="MR270"/>
 <element name="JP5" library="TiLDA Mk4 Parts" package="1X08_LOCK" value="1x08" x="18" y="75" locked="yes" rot="MR195">
 <attribute name="DNP" value="Y" x="18" y="75" size="1.778" layer="28" rot="MR195" display="off"/>
@@
 <attribute name="DNP" value="Y" x="-18" y="75" size="1.778" layer="28" rot="MR345" display="off"/>
 </element>
-<element name="U1" library="TiLDA Mk4 Parts" package="USB-AB-MICRO-SMD_LWK" value="ZX62-AB-5PA(11)" x="10.4" y="75.5" rot="MR274"/>
+<element name="U1" library="TiLDA Mk4 Parts" package="USB-AB-MICRO-SMD_LWK" value="ZX62-B-5PA(33)" x="10.4" y="75.5" rot="MR274"/>
 <element name="J1" library="TiLDA Mk4 Parts" package="MSIM-MOLEX-LWK" value="78723-1001" x="57" y="21" rot="MR180"/>
 <element name="J4" library="TiLDA Mk4 Parts" package="GSM-ANTENNA" value="GSM-COIL-ANT" x="56.5" y="36" rot="MR0"/>
@@
 <attribute name="TP_SIGNAL_NAME" value="!HIB" x="-7.6" y="60.7" size="1.016" layer="28" ratio="15" rot="MR0" display="off"/>
 </element>
-<element name="X1" library="TiLDA Mk4 Parts" package="RESONATOR_EPSON_FC_145" value="FC-135R 32.768KHZ 9PF" x="-5.6" y="64.25" rot="MR180"/>
-<element name="X2" library="TiLDA Mk4 Parts" package="CRYSTAL-3.2-2.5" value="NX3225GA-25.000M-STD-CRG-2" x="3.25" y="67.75" rot="MR90"/>
+<element name="X1" library="TiLDA Mk4 Parts" package="RESONATOR_EPSON_FC_145" value="ABS07-32.768KHZ-T" x="-5.6" y="64.25" rot="MR180"/>
+<element name="X2" library="TiLDA Mk4 Parts" package="CRYSTAL-3.2-2.5" value="ABM8G-25.000MHZ-B4Y-T" x="3.25" y="67.75" rot="MR90"/>
 <element name="R6" library="TiLDA Mk4 Parts" package="R0402-SMALLER" value="0402/2K/5%" x="3.75" y="63.75" rot="MR90"/>
 <element name="C16" library="TiLDA Mk4 Parts" package="C0402-SMALLER" value="0402/12p/50V/C0G" x="2.25" y="65.25" rot="MR180"/>
@@
 <attribute name="DNP" value="Y" x="-51" y="39" size="1.778" layer="28" rot="MR0" display="off"/>
 </element>
-<element name="ANT1" library="TiLDA Mk4 Parts" package="2450AT18D0100-RIGHT" value="24509AT1BD100" x="-48.25" y="68" rot="MR160"/>
-<element name="ANT2" library="TiLDA Mk4 Parts" package="2450AT18D0100" value="24509AT1BD100" x="48.25" y="68" rot="MR20"/>
+<element name="ANT1" library="TiLDA Mk4 Parts" package="2450AT18D0100-RIGHT" value="2450AT18D0100" x="-48.25" y="68" rot="MR160"/>
+<element name="ANT2" library="TiLDA Mk4 Parts" package="2450AT18D0100" value="2450AT18D0100" x="48.25" y="68" rot="MR20"/>
 <element name="C48" library="TiLDA Mk4 Parts" package="C0402-SMALLER" value="0402/22p/10V/X5R" x="41.5" y="52.5" rot="MR270"/>
 <element name="C49" library="TiLDA Mk4 Parts" package="C0402-SMALLER" value="0402/22p/10V/X5R" x="38.5" y="52.5" rot="MR270"/>
@@
 <element name="R55" library="TiLDA Mk4 Parts" package="R0402-SMALLER" value="0402/10K/5%" x="27.75" y="49.75" rot="MR180"/>
 <element name="R56" library="TiLDA Mk4 Parts" package="R0402-SMALLER" value="0402/10K/5%" x="34.25" y="59.5" rot="MR180"/>
-<element name="IC13" library="TiLDA Mk4 Parts" package="VSON-8" value="TPA2066D1" x="-34.5" y="27.25" rot="MR0"/>
+<element name="IC13" library="TiLDA Mk4 Parts" package="VSON-8" value="TPA2006D1" x="-34.5" y="27.25" rot="MR0"/>
 <element name="R57" library="TiLDA Mk4 Parts" package="R0402-SMALLER" value="0402/150K/1%" x="-31.25" y="27.25" rot="MR0"/>
 <element name="R58" library="TiLDA Mk4 Parts" package="R0402-SMALLER" value="0402/150K/1%" x="-31.25" y="26.25" rot="MR0"/>
@@
 <attribute name="DNP" value="Y" x="-34.5" y="31" size="1.778" layer="28" rot="MR0" display="off"/>
 </element>
+<element name="BATT" library="TiLDA Mk4 Parts" package="BATTERY-32X50" value="1000mAh JST-PH" x="-0.5" y="12" rot="R90"/>
 </elements>
 <signals>
 <signal name="GND">
-<contactref element="OUTLINE1" pad="GND"/>
+<contactref element="PCB" pad="GND"/>
 <contactref element="C45" pad="1"/>
 <contactref element="C38" pad="1"/>
@@
 <via x="-38" y="53" extent="1-16" drill="0.3"/>
 <via x="-30.25" y="49" extent="1-16" drill="0.3"/>
-<contactref element="JP1" pad="1"/>
+<contactref element="J5" pad="1"/>
 <via x="19.5" y="14.75" extent="1-16" drill="0.3"/>
 <via x="21" y="13.5" extent="1-16" drill="0.3"/>
@@
 </signal>
 <signal name="VBAT">
-<contactref element="JP1" pad="2"/>
+<contactref element="J5" pad="2"/>
 <contactref element="IC8" pad="13"/>
 <contactref element="IC8" pad="14"/>
@@
 </signal>
 <signal name="3V3">
-<contactref element="OUTLINE1" pad="3V3"/>
+<contactref element="PCB" pad="3V3"/>
 <contactref element="SW1" pad="COM"/>
 <contactref element="C38" pad="2"/>
@@
 </signal>
 <signal name="V_UNREG">
-<contactref element="OUTLINE1" pad="VBATT"/>
+<contactref element="PCB" pad="VBATT"/>
 <contactref element="IC8" pad="16"/>
 <contactref element="IC8" pad="15"/>
@@
 </signal>
 <signal name="CH1">
-<contactref element="OUTLINE1" pad="CH4"/>
+<contactref element="PCB" pad="CH4"/>
 </signal>
 <signal name="CH2">
-<contactref element="OUTLINE1" pad="CH3"/>
+<contactref element="PCB" pad="CH3"/>
 </signal>
 <signal name="CH3">
-<contactref element="OUTLINE1" pad="CH2"/>
+<contactref element="PCB" pad="CH2"/>
 </signal>
 <signal name="CH4">
-<contactref element="OUTLINE1" pad="CH1"/>
+<contactref element="PCB" pad="CH1"/>
 </signal>
 <signal name="FET_OUT">
-<contactref element="OUTLINE1" pad="FET"/>
+<contactref element="PCB" pad="FET"/>
 <contactref element="LED5" pad="K"/>
 <contactref element="Q2" pad="3"/>
@@
 </signal>
 <signal name="I2C2_SDA">
-<contactref element="OUTLINE1" pad="SDA"/>
+<contactref element="PCB" pad="SDA"/>
 <contactref element="R23" pad="1"/>
 <wire x1="43.96194375" y1="5.8333125" x2="-1" y2="56.5" width="0" layer="19" extent="16-16"/>
 </signal>
 <signal name="I2C2_SCL">
-<contactref element="OUTLINE1" pad="SCL"/>
+<contactref element="PCB" pad="SCL"/>
 <contactref element="R24" pad="1"/>
 <wire x1="37.79828125" y1="4.38555625" x2="-1" y2="55.5" width="0" layer="19" extent="16-16"/>
